File: PCB/GSM-GPS-tryout/stm32.sch (KiCad schematic (older format))
At the start: 38 parts

Commit message: update,
Parts:
- gave numbers to parts that had none: 38

Commit message: update,
Parts:
- removed D2: RED, LED_SMD:LED_0805_2012Metric_Pad1.15x1.40mm_HandSolder, symbol Device:LED
- removed J1: Conn_01x04, Connector_PinHeader_1.27mm:PinHeader_1x04_P1.27mm_Vertical, symbol Connector_Generic:Conn_01x04
- removed SW1: SW_SPST, Button_Switch_THT:SW_PUSH_6mm_H4.3mm, symbol Switch:SW_SPST
- added D12: 5V_STATUS, LED_SMD:LED_0805_2012Metric_Pad1.15x1.40mm_HandSolder, symbol Device:LED
- added D13: 3V3_STATUS, LED_SMD:LED_0805_2012Metric_Pad1.15x1.40mm_HandSolder, symbol Device:LED
- added D2: 1N5819, Diode_THT:D_DO-41_SOD81_P10.16mm_Horizontal, symbol Diode:1N5819
- added J1: Conn_01x02, Connector_PinHeader_2.54mm:PinHeader_1x02_P2.54mm_Vertical, symbol Connector_Generic:Conn_01x02
- added R32: 510, Resistor_SMD:R_0805_2012Metric_Pad1.15x1.40mm_HandSolder, symbol Device:R
- added SW1: SW_Push, symbol Switch:SW_Push
- C1: value 10u -> 10u (25V)
- C3, C4, C5, C6, C7, C8: footprint Capacitor_SMD:C_0603_1608Metric_Pad1.05x0.95mm_HandSolder -> Capacitor_SMD:C_0805_2012Metric_Pad1.15x1.40mm_HandSolder
- D1: value LED -> PB3_LED
- D3: value RED -> STM_PWR_STATUS
- J4: value Conn_02x04_Row_Letter_First -> SWD_CONN
- R2: value 510 -> 1k
- R4: value R -> 10k
- U1: value AMS1117-1.8 -> AMS1117-3.3
Connections:
- net labels added: +3V3, PB2, PB8
- net labels removed: VIN
- wire segments 168 -> 177
- no-connect marks 8 -> 5
Other:
- note added: "NRST is not connected \nin the origional design"
- note added: "the pin assignment try to fit \nwith the waveshare SWD stick"
- note removed: "Assuming:\n\nVIN = +5V\nVDD = +1.8V\n\n"
- note removed: "SWO is not connected \nin the origional design"
- note removed: "TERMINAL FOR \nCONNECTING TO BATTERY"
- note removed: "add additional led for incidate the power status\nfor both 5V and 3.3V"
- note removed: "additional pcb jumper for \npower measurment in \norigional design"
- note removed: "replace the combination of Vin -> 5V -> 3.3V \ndirectly to Vin -> 3.3V"
- note removed: "the pin assignment is try to fit \nwith the waveshare SWD stick"
