File: PCB/GSM-GPS-tryout/GSM-GPS-tryout.sch (KiCad schematic (older format))
At the start: 12 parts

Commit message: update,
Parts:
- added BEAD1: L1, symbol Device:L
- added C11, C23, C24, C7: 100n, Capacitor_SMD:C_0603_1608Metric_Pad1.05x0.95mm_HandSolder, symbol Device:C
- added C22, C25: 10u, Capacitor_SMD:CP_Elec_3x5.4, symbol Device:CP
- added D1: LED, LED_SMD:LED_0805_2012Metric_Pad1.15x1.40mm_HandSolder, symbol Device:LED
- added D2, D3: RED, LED_SMD:LED_0805_2012Metric_Pad1.15x1.40mm_HandSolder, symbol Device:LED
- added J1: Conn_01x04, Connector_PinHeader_1.27mm:PinHeader_1x04_P1.27mm_Vertical, symbol Connector_Generic:Conn_01x04
- added J4: Conn_02x04_Row_Letter_First, Connector_PinHeader_2.54mm:PinHeader_2x04_P2.54mm_Vertical, symbol Connector_Generic:Conn_02x04_Row_Letter_First
- added J5: Conn_01x02, Connector_PinHeader_2.54mm:PinHeader_1x02_P2.54mm_Vertical, symbol Connector_Generic:Conn_01x02
- added JP1, JP10, JP11, JP13, JP2, JP3, JP4: Jumper, Jumper:SolderJumper-2_P1.3mm_Bridged_Pad1.0x1.5mm, symbol Device:Jumper
- added R1, R2, R22: 510, Resistor_SMD:R_0805_2012Metric_Pad1.15x1.40mm_HandSolder, symbol Device:R
- added R3: R, Resistor_SMD:R_0805_2012Metric_Pad1.15x1.40mm_HandSolder, symbol Device:R
- added SW1: SW_SPST, Button_Switch_THT:SW_PUSH_6mm_H4.3mm, symbol Switch:SW_SPST
- added U6: AMS1117-1.8, Package_TO_SOT_SMD:SOT-223-3_TabPin2, symbol Regulator_Linear:AMS1117-1.8
- C12, C13: renamed from C?; value C -> 4.3p; footprint (none) -> Capacitor_SMD:C_0603_1608Metric_Pad1.05x0.95mm_HandSolder
- J2, J3, J6, J7: renamed from J?; footprint (none) -> Connector_PinHeader_1.27mm:PinHeader_1x08_P1.27mm_Vertical
- JP5, JP6, JP7, JP8: renamed from JP?; footprint (none) -> Jumper:SolderJumper-2_P1.3mm_Bridged_Pad1.0x1.5mm
- Y1: renamed from Y?; value Crystal -> 32.768K; footprint (none) -> Crystal:Crystal_HC49-4H_Vertical
- gave numbers to parts that had none: 1
Connections:
- net labels added: +3.3V, +5V, AVDD, BOOT0, NRST, PA0, PA1, PA10, PA11, PA12, PA13, PA14, PA15, PA2, PA3, PA4, PA5, PA6, PA7, PA8, PA9, PB0, PB1, PB3, PB4, PB5, PB6, PB7, SWCLK, SWDIO, VCP_RX, VCP_TX, VDD, VIN
- wire segments 24 -> 168
- no-connect marks 0 -> 8
Other:
- note added: "Assuming:\n\nVIN = +5V\nVDD = +1.8V\n\n"
- note added: "INCIDATORS BANK"
- note added: "IO BANK CONFIGURATION"
- note added: "MCO neglected"
- note added: "SWIM"
- note added: "SWIM is not connected \ndue to not necessary"
- note added: "SWO is not connected \nin the origional design"
- note added: "TERMINAL FOR \nCONNECTING TO BATTERY"
- note added: "add additional led for incidate the power status\nfor both 5V and 3.3V"
- note added: "additional pcb jumper for \npower measurment in \norigional design"
- note added: "replace the combination of Vin -> 5V -> 3.3V \ndirectly to Vin -> 3.3V"
- note added: "the pin assignment is try to fit \nwith the waveshare SWD stick"
- moved on the sheet: U1

Commit message: update,
Parts:
- removed BEAD1: L1, symbol Device:L
- removed C11, C23, C24, C7: 100n, Capacitor_SMD:C_0603_1608Metric_Pad1.05x0.95mm_HandSolder, symbol Device:C
- removed C12, C13: 4.3p, Capacitor_SMD:C_0603_1608Metric_Pad1.05x0.95mm_HandSolder, symbol Device:C
- removed C22, C25: 10u, Capacitor_SMD:CP_Elec_3x5.4, symbol Device:CP
- removed D1: LED, LED_SMD:LED_0805_2012Metric_Pad1.15x1.40mm_HandSolder, symbol Device:LED
- removed D2, D3: RED, LED_SMD:LED_0805_2012Metric_Pad1.15x1.40mm_HandSolder, symbol Device:LED
- removed J1: Conn_01x04, Connector_PinHeader_1.27mm:PinHeader_1x04_P1.27mm_Vertical, symbol Connector_Generic:Conn_01x04
- removed J2, J3, J6, J7: Conn_01x08, Connector_PinHeader_1.27mm:PinHeader_1x08_P1.27mm_Vertical, symbol Connector_Generic:Conn_01x08
- removed J4: Conn_02x04_Row_Letter_First, Connector_PinHeader_2.54mm:PinHeader_2x04_P2.54mm_Vertical, symbol Connector_Generic:Conn_02x04_Row_Letter_First
- removed J5: Conn_01x02, Connector_PinHeader_2.54mm:PinHeader_1x02_P2.54mm_Vertical, symbol Connector_Generic:Conn_01x02
- removed JP1, JP10, JP11, JP13, JP2, JP3, JP4, JP5, JP6, JP7, JP8: Jumper, Jumper:SolderJumper-2_P1.3mm_Bridged_Pad1.0x1.5mm, symbol Device:Jumper
- removed R1, R2, R22: 510, Resistor_SMD:R_0805_2012Metric_Pad1.15x1.40mm_HandSolder, symbol Device:R
- removed R3: R, Resistor_SMD:R_0805_2012Metric_Pad1.15x1.40mm_HandSolder, symbol Device:R
- removed SW1: SW_SPST, Button_Switch_THT:SW_PUSH_6mm_H4.3mm, symbol Switch:SW_SPST
- removed U1: STM32L011K4Tx, Package_QFP:LQFP-32_7x7mm_P0.8mm, symbol MCU_ST_STM32L0:STM32L011K4Tx
- removed U6: AMS1117-1.8, Package_TO_SOT_SMD:SOT-223-3_TabPin2, symbol Regulator_Linear:AMS1117-1.8
- removed Y1: 32.768K, Crystal:Crystal_HC49-4H_Vertical, symbol Device:Crystal
Connections:
- net labels removed: +3.3V, +5V, AVDD, BOOT0, GND, NRST, PA0, PA1, PA10, PA11, PA12, PA13, PA14, PA15, PA2, PA3, PA4, PA5, PA6, PA7, PA8, PA9, PB0, PB1, PB3, PB4, PB5, PB6, PB7, PC14, PC15, SWCLK, SWDIO, VCP_RX, VCP_TX, VDD, VIN
- wire segments 168 -> 0
- no-connect marks 8 -> 0
Other:
- note removed: "Assuming:\n\nVIN = +5V\nVDD = +1.8V\n\n"
- note removed: "INCIDATORS BANK"
- note removed: "IO BANK CONFIGURATION"
- note removed: "MCO neglected"
- note removed: "SWIM"
- note removed: "SWIM is not connected \ndue to not necessary"
- note removed: "SWO is not connected \nin the origional design"
- note removed: "TERMINAL FOR \nCONNECTING TO BATTERY"
- note removed: "add additional led for incidate the power status\nfor both 5V and 3.3V"
- note removed: "additional pcb jumper for \npower measurment in \norigional design"
- note removed: "replace the combination of Vin -> 5V -> 3.3V \ndirectly to Vin -> 3.3V"
- note removed: "the pin assignment is try to fit \nwith the waveshare SWD stick"

Commit message: update,
Changed lines of the file:
@@
 $Descr A3 16535 11693
 encoding utf-8
-Sheet 1 3
+Sheet 1 4
 Title ""
 Date ""
@@
 F1 "SIM800C.sch" 50
 $EndSheet
+$Sheet
+S 4250 850  1550 950
+U 5BBADC15
+F0 "ublox-gps" 50
+F1 "ublox-gps.sch" 50
+$EndSheet
 $EndSCHEMATC
