File: PCB/GSM-GPS-tryout/SIM800C.sch (KiCad schematic (older format))
At the start: 3 parts

Commit message: update,
Parts:
- gave numbers to parts that had none: 3
Changed lines of the file:
@@
 $EndDescr
 $Comp
-L SIM_COM:SIM800C U?
+L SIM_COM:SIM800C U3
 U 1 1 5BB865BD
 P 4800 2800
-F 0 "U?" H 5841 2846 50  0000 L CNN
+F 0 "U3" H 5841 2846 50  0000 L CNN
 F 1 "SIM800C" H 5841 2755 50  0000 L CNN
 F 2 "SIMCOM_modules:SIM800C" H 4800 2800 50  0001 C CNN
@@
 $EndComp
 $Comp
-L Connector:SIM_Card J?
+L Connector:SIM_Card J8
 U 1 1 5BB865F3
 P 9000 1950
-F 0 "J?" H 9629 2050 50  0000 L CNN
+F 0 "J8" H 9629 2050 50  0000 L CNN
 F 1 "SIM_Card" H 9629 1959 50  0000 L CNN
 F 2 "" H 9000 2300 50  0001 C CNN
@@
 $EndComp
 $Comp
-L Device:Antenna_Shield AE?
+L Device:Antenna_Shield AE1
 U 1 1 5BB86668
 P 7600 3300
-F 0 "AE?" H 7740 3341 50  0000 L CNN
+F 0 "AE1" H 7740 3341 50  0000 L CNN
 F 1 "Antenna_Shield" H 7740 3250 50  0000 L CNN
 F 2 "" H 7600 3400 50  0001 C CNN

Commit message: update,
Parts:
- removed AE1: Antenna_Shield, symbol Device:Antenna_Shield
- removed J8: SIM_Card, symbol Connector:SIM_Card
- added C? (x2): 10u, symbol Device:C
- added C?: 100u, symbol Device:CP
- added C?: 33p, symbol Device:C
- added C?: 10p, symbol Device:C
- added C?: 10u, symbol Device:CP
- added C?: 0.1u, symbol Device:C
- added C?: 1u, symbol Device:C
- added D?: MMSZ5231BT1G, SOD123, symbol Device:D_Schottky
- added D?: BLUE, symbol Device:LED
- added D?: GREEN, symbol Device:LED
- added D? (x2): D_Zener, symbol Device:D_Zener
- added D_CHRG: O, symbol Device:LED
- added D_DONE: G, symbol Device:LED
- added J?: USB_B_Micro, symbol Connector:USB_B_Micro
- added J? (x2): Conn_01x02, symbol Connector_Generic:Conn_01x02
- added J?: Conn_Coaxial, symbol Connector:Conn_Coaxial
- added J?: SIM_COM_MODULE, symbol Connector_Generic:Conn_01x08
- added J?: TO_DTE (+3V3), symbol Connector_Generic:Conn_01x08
- added J?: TO_DTE (+3V3), symbol Connector_Generic:Conn_01x05
- added JP?: Jumper, symbol Device:Jumper
- added Q?: Q_NPN_BCE, symbol Device:Q_NPN_BCE
- added R?: 2k, symbol Device:R
- added R?: 470, symbol Device:R
- added R? (x9): 1k, symbol Device:R
- added R?: 10k, symbol Device:R
- added R? (x2): 4.7k, symbol Device:R
- added R?: 47k, symbol Device:R
- added R? (x3): R, symbol Device:R
- added R? (x3): 5.6k, symbol Device:R
- added R? (x3): 51, symbol Device:R
- added SW?: SW_SPST, symbol Switch:SW_SPST
- added U?: MCP73831-2-OT, Package_TO_SOT_SMD:SOT-23-5, symbol Battery_Management:MCP73831-2-OT
- added U?: SMF05C, symbol smf05c.lib:SMF05C
- added U?: Molex 91228 SIM card holder, symbol SIM_SLOT:SIM_CARD
Connections:
- net labels added: +1V8, +2V8, +5V, +BATT, GND, GSM_ANT, MIC1N, MIC1P, NETLIGHT, PWRKEY, SIM800C_ADC, SIMCLK, SIMCOM_PWRKEY, SIMDATA, SIMDET, SIMRST, SPK1N, SPK1P, UART1_CTS_3V3, UART1_DCD_3V3, UART1_DTR_3V3, UART1_RI_3V3, UART1_RTS_3V3, UART1_RXD_3V3, UART1_TXD_3V3, USB_DN, USB_DP, USB_GND, USB_ID, USB_VBUS
- wire segments 0 -> 232
Other:
- note added: "4.1. Power Supply"
- note added: "COMMENTS\n\ntry to align PIN1 the GROUND\n\n4.1.1. Power Supply Pin\nThe PCB traces from the VBAT pins to the power supply must be wide enough (at least 60mil) to decrease voltage drops\nThe power IC and the bypass capacitor should be placed to the module as close as possible.\n\n4.2.1. Power on SIM800C\nCustomer can power on SIM800C by pulling down the PWRKEY pin for at least 1 second and releas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"
- note added: "IO PORT BANK"
- note added: "POWER SUPPLY\nAND GOUND"
- note added: "SIM CARD HOLDER\n"
- note added: "STATUS LED\n"
- note added: "USB source\nand charging circuit"
- note added: "VBAT input, a 100uF Tantalum capacitor (C A low ESR) and \na 1uF~10uF Ceramics capacitor C B are strongly recommended."
- note added: "from SIM800C_Hardware_Design_V1.00"

Commit message: update,
Parts:
- removed J?: USB_B_Micro, symbol Connector:USB_B_Micro
- removed R?: 47k, symbol Device:R
- removed SW?: SW_SPST, symbol Switch:SW_SPST
- added C21: 10u, symbol Device:C
- added J16: TO_DTE (+3V3), symbol Connector_Generic:Conn_01x02
- added J17: Conn_Coaxial, symbol Connector:Conn_Coaxial
- added J8: Conn_01x04, symbol Connector_Generic:Conn_01x04
- added JP12: Jumper, Jumper:SolderJumper-2_P1.3mm_Bridged_Pad1.0x1.5mm, symbol Device:Jumper
- added SW2: SW_Push, symbol Switch:SW_Push
- C10, C12, C13, C14, C16, C9: renamed from C?; footprint (none) -> Capacitor_SMD:C_0805_2012Metric_Pad1.15x1.40mm_HandSolder
- C11: renamed from C?; footprint (none) -> Capacitor_SMD:CP_Elec_4x5.3
- D4, D5: renamed from D?; footprint (none) -> LED_SMD:LED_0805_2012Metric_Castellated
- D6: renamed from D?; footprint SOD123 -> Diode_SMD:D_SOD-123
- JP13: renamed from JP?; footprint (none) -> Jumper:SolderJumper-2_P1.3mm_Bridged_Pad1.0x1.5mm
- Q1: renamed from Q?; value Q_NPN_BCE -> SS9013
- R10: renamed from R?; value 4.7k -> 1k; footprint (none) -> Resistor_SMD:R_0805_2012Metric_Pad1.15x1.40mm_HandSolder
- R12, R13, R14, R15, R16, R17, R18, R19, R20, R21, R22, R23, R24, R25, R26, R27, R28, R5, R6, R7, R8, R9: renamed from R?; footprint (none) -> Resistor_SMD:R_0805_2012Metric_Pad1.15x1.40mm_HandSolder
- U5: renamed from U?; footprint (none) -> Silicon-Standard:SC70-6
- gave numbers to parts that had none: 11
- renumbered D_CHRG to D_CHRG1, D_DONE to D_DONE1
Connections:
- net labels added: BT_ANT, SIMVDD, UART2_RXD, UART2_TXD
- net labels removed: +1V8, MIC1N, MIC1P, SIM800C_ADC, SPK1N, SPK1P
- wire segments 232 -> 237
- no-connect marks 0 -> 4
Other:
- note added: "ANTENNA FARM"
- note added: "SIM\nPRESENT"

Commit message: update,
Parts:
- removed J12: TO_DTE (+3V3), symbol Connector_Generic:Conn_01x05
- added J12: USB_B_Mini, symbol Connector:USB_B_Mini
Connections:
- net labels removed: USB_ID
- wire segments 237 -> 239
- no-connect marks 4 -> 5
Changed lines of the file:
@@
 	14000 7100 14200 7100
-$Comp
-L Connector_Generic:Conn_01x05 J12
-U 1 1 5C0E8B34
-P 15000 5450
-F 0 "J12" H 14919 5025 50  0000 C CNN
-F 1 "TO_DTE (+3V3)" H 14919 5116 50  0000 C CNN
-F 2 "" H 15000 5450 50  0001 C CNN
-F 3 "~" H 15000 5450 50  0001 C CNN
-	1    15000 5450
-	1    0    0    1
-$EndComp
 $Comp
 L power:GND #PWR0153
@@
 $EndComp
 Text Label 13450 5450 0    50   ~ 0
+USB_DN
+Text Label 13450 5350 0    50   ~ 0
 USB_DP
-Text Label 13450 5350 0    50   ~ 0
-USB_DN
-Text Label 13450 5250 0    50   ~ 0
+Text Label 13450 5150 0    50   ~ 0
 USB_VBUS
 $Comp
@@
 $EndComp
 Wire Wire Line
-	14250 4450 14250 4750
-Wire Wire Line
-	14250 5250 14800 5250
+	14250 5150 14800 5150
 $Comp
 L Device:C C16
@@
 	14300 4750 14250 4750
 Connection ~ 14250 4750
-Wire Wire Line
-	14250 4750 14250 5250
 $Comp
 L power:GND #PWR0155
@@
 Wire Wire Line
 	14800 4750 14600 4750
-Text Label 13450 5550 0    50   ~ 0
-USB_ID
 Text Label 10100 3000 3    50   ~ 0
 USB_DN
@@
 	10300 3000 10300 3800
 Wire Wire Line
-	13450 5250 14250 5250
-Connection ~ 14250 5250
-Wire Wire Line
-	13450 5550 14800 5550
+	13450 5150 14250 5150
+Connection ~ 14250 5150
 Text Label 13500 6250 0    50   ~ 0
 USB_GND
@@
 Wire Wire Line
 	13950 6250 13950 6350
-Wire Wire Line
-	14700 5650 14800 5650
 Connection ~ 13950 6250
-Wire Wire Line
-	14700 5650 14700 6250
 $Comp
 L Device:D_Zener D7
@@
 	14600 6000 14600 6250
 Connection ~ 14600 6250
-Wire Wire Line
-	14600 6250 14700 6250
 Wire Wire Line
 	14250 5700 14250 5450
@@
 Text Notes 1900 9750 0    50   ~ 0
 SIM\nPRESENT
+$Comp
+L Connector:USB_B_Mini J12
+U 1 1 5C0F2B62
+P 15100 5350
+F 0 "J12" H 14871 5341 50  0000 R CNN
+F 1 "USB_B_Mini" H 14871 5250 50  0000 R CNN
+F 2 "" H 15250 5300 50  0001 C CNN
+F 3 "~" H 15250 5300 50  0001 C CNN
+	1    15100 5350
+	-1   0    0    -1
+$EndComp
+Wire Wire Line
+	14250 4750 14250 5150
+Wire Wire Line
+	15100 5750 15100 5950
+Wire Wire Line
+	14250 4650 14250 4750
+Wire Wire Line
+	14250 4450 14250 4750
+Wire Wire Line
+	15200 5750 15200 5950
+Wire Wire Line
+	15200 5950 15100 5950
+Connection ~ 15100 5950
+Wire Wire Line
+	15100 5950 15100 6250
+Wire Wire Line
+	14600 6250 15100 6250
+NoConn ~ 14800 5550
 $EndSCHEMATC
