File: PCB/GSM-GPS-tryout.kicad_pcb (KiCad board)
At the start: 2 copper layers, 37 parts, among them J1 Conn_01x04, J2 Conn_01x08, J3 Conn_01x08, J4 Conn_02x04_Row_Letter_First, J5 Conn_01x02, J6 Conn_01x08, J7 Conn_01x08, SW1 SW_SPST, U1 STM32L011K4Tx, U6 AMS1117-1.8, Y1 32.768K

Commit message: updte
Parts:
- removed C23, C24: 100n, Capacitor_SMD:C_0603_1608Metric_Pad1.05x0.95mm_HandSolder
- removed C25: 10u, Capacitor_SMD:CP_Elec_3x5.4
- removed R22: 510, Resistor_SMD:R_0805_2012Metric_Pad1.15x1.40mm_HandSolder
- added BT1: MS621F, Battery:BatteryHolder_Seiko_MS621F, F.Cu at (147.4, 63.4)
- added C1: 56u, Capacitor_SMD:CP_Elec_3x5.4, F.Cu at (194.3, 17.4)
- added C10: C33pf, Capacitor_SMD:C_0805_2012Metric_Pad1.15x1.40mm_HandSolder, F.Cu at (165.1, 31.9)
- added C14: C106, Capacitor_SMD:C_0805_2012Metric_Pad1.15x1.40mm_HandSolder, F.Cu at (165.1, 39.7)
- added C15: C106, Capacitor_SMD:C_0805_2012Metric_Pad1.15x1.40mm_HandSolder, F.Cu at (163.3, 44.1)
- added C16: CP220uf,16V, Capacitor_SMD:CP_Elec_6.3x7.7, F.Cu at (129.5, 39.7)
- added C17: C104, Capacitor_SMD:C_0603_1608Metric_Pad1.05x0.95mm_HandSolder, F.Cu at (137.3, 44.5)
- added C18: C106, Capacitor_SMD:C_0603_1608Metric_Pad1.05x0.95mm_HandSolder, F.Cu at (134.0, 44.5)
- added C19: C105, Capacitor_SMD:C_0603_1608Metric_Pad1.05x0.95mm_HandSolder, F.Cu at (155.9, 55.3)
- added C2: 10u, Capacitor_SMD:CP_Elec_3x5.4, F.Cu at (194.3, 21.3)
- added C20: C106, Capacitor_SMD:C_0603_1608Metric_Pad1.05x0.95mm_HandSolder, F.Cu at (144.5, 58.8)
- added C21: C104, Capacitor_SMD:C_0603_1608Metric_Pad1.05x0.95mm_HandSolder, F.Cu at (150.3, 60.9)
- added C3: C4.7pf, Capacitor_SMD:C_0805_2012Metric_Pad1.15x1.40mm_HandSolder, F.Cu at (197.1, 24.2)
- added C4: C4.7pf, Capacitor_SMD:C_0805_2012Metric_Pad1.15x1.40mm_HandSolder, F.Cu at (199.1, 16.5)
- added C5: C104, Capacitor_SMD:C_0805_2012Metric_Pad1.15x1.40mm_HandSolder, F.Cu at (186.9, 26.7)
- added C6: C104, Capacitor_SMD:C_0805_2012Metric_Pad1.15x1.40mm_HandSolder, F.Cu at (194.4, 26.1)
- added C8: C104, Capacitor_SMD:C_0805_2012Metric_Pad1.15x1.40mm_HandSolder, F.Cu at (199.1, 20.4)
- added C9: C33pf, Capacitor_SMD:C_0805_2012Metric_Pad1.15x1.40mm_HandSolder, F.Cu at (165.1, 37.7)
- added D10: LED_GREEN, LED_SMD:LED_0805_2012Metric_Castellated, F.Cu at (130.6, 66.0)
- added D11: SD_1N5817_SS12, Diode_SMD:D_1206_3216Metric_Pad1.42x1.75mm_HandSolder, F.Cu at (152.9, 49.7)
- added D12: 5V_STATUS, LED_SMD:LED_0805_2012Metric_Pad1.15x1.40mm_HandSolder, F.Cu at (163.0, 49.5)
- added D4: LED_GREEN, LED_SMD:LED_0805_2012Metric_Castellated, F.Cu at (183.1, 26.7)
- added D5: LED_GREEN, LED_SMD:LED_0805_2012Metric_Castellated, F.Cu at (168.8, 26.9)
- added D6: LED_GREEN, LED_SMD:LED_0805_2012Metric_Castellated, F.Cu at (168.8, 28.9)
- added D7: ZD_4V7, Diode_SMD:D_1206_3216Metric_Pad1.42x1.75mm_HandSolder, F.Cu at (159.0, 44.3)
- added D8: LED_RED, LED_SMD:LED_0805_2012Metric_Castellated, F.Cu at (173.7, 24.1)
- added D9: LED_BLUE, LED_SMD:LED_0805_2012Metric_Castellated, F.Cu at (126.8, 66.0)
- added FB1: Ferrite_Bead_Small, w_smd_inductors:inductor_smd_0805, F.Cu at (202.5, 16.6)
- added J10: Conn_01x05, Connector_PinHeader_2.54mm:PinHeader_1x05_P2.54mm_Vertical, F.Cu at (165.1, 17.3)
- added J11: Conn_01x02, Connector_PinHeader_2.54mm:PinHeader_1x02_P2.54mm_Vertical, F.Cu at (176.3, 17.3)
- added J15: Conn_01x04, Connector_PinHeader_2.54mm:PinHeader_1x04_P2.54mm_Vertical, F.Cu at (141.0, 50.4)
- added J8: Conn_01x05, Connector_PinHeader_2.54mm:PinHeader_1x05_P2.54mm_Vertical, F.Cu at (161.4, 17.3)
- added J9: Conn_01x05, Connector_PinHeader_2.54mm:PinHeader_1x05_P2.54mm_Vertical, F.Cu at (161.4, 31.1)
- added JP12: Jumper, Jumper:SolderJumper-2_P1.3mm_Bridged_Pad1.0x1.5mm, F.Cu at (201.3, 25.2)
- added JP14: Jumper_NC_Small, Jumper:SolderJumper-2_P1.3mm_Bridged_Pad1.0x1.5mm, F.Cu at (200.6, 22.6)
- added JP15: Jumper_NO_Small, Jumper:SolderJumper-2_P1.3mm_Open_TrianglePad1.0x1.5mm, F.Cu at (166.1, 52.4)
- added JP16: Jumper_NO_Small, Jumper:SolderJumper-2_P1.3mm_Open_TrianglePad1.0x1.5mm, F.Cu at (166.6, 49.8)
- added JP17: Jumper, Jumper:SolderJumper-2_P1.3mm_Bridged_Pad1.0x1.5mm, F.Cu at (198.0, 26.4)
- added JP9: Jumper_NO_Small, Jumper:SolderJumper-2_P1.3mm_Open_TrianglePad1.0x1.5mm, F.Cu at (162.8, 51.8)
- added L2: 22u, w_smd_inductors:inductor_smd_0805, F.Cu at (154.0, 59.3)
- added R10: R220, Resistor_SMD:R_0805_2012Metric_Pad1.15x1.40mm_HandSolder, F.Cu at (172.6, 29.9)
- added R11: R102, Resistor_SMD:R_0805_2012Metric_Pad1.15x1.40mm_HandSolder, F.Cu at (173.6, 26.0)
- added R12: R_Small, Resistor_SMD:R_0805_2012Metric_Pad1.15x1.40mm_HandSolder, F.Cu at (165.1, 35.8)
- added R13: R433, Resistor_SMD:R_0805_2012Metric_Pad1.15x1.40mm_HandSolder, F.Cu at (168.9, 32.8)
- added R14: R104, Resistor_SMD:R_0805_2012Metric_Pad1.15x1.40mm_HandSolder, F.Cu at (165.1, 33.8)
- added R15: R471, Resistor_SMD:R_0805_2012Metric_Pad1.15x1.40mm_HandSolder, F.Cu at (168.9, 34.7)
- added R16: R102, Resistor_SMD:R_0805_2012Metric_Pad1.15x1.40mm_HandSolder, F.Cu at (168.9, 30.8)
- added R17: R102, Resistor_SMD:R_0805_2012Metric_Pad1.15x1.40mm_HandSolder, F.Cu at (134.4, 66.1)
- added R18: R220, Resistor_SMD:R_0805_2012Metric_Pad1.15x1.40mm_HandSolder, F.Cu at (150.5, 59.2)
- added R19: R102, Resistor_SMD:R_0805_2012Metric_Pad1.15x1.40mm_HandSolder, F.Cu at (148.4, 57.1)
- added R20: R102, Resistor_SMD:R_0805_2012Metric_Pad1.15x1.40mm_HandSolder, F.Cu at (144.7, 57.1)
- added R4: R511, Resistor_SMD:R_0805_2012Metric_Pad1.15x1.40mm_HandSolder, F.Cu at (190.7, 26.7)
- added R5: R511, Resistor_SMD:R_0805_2012Metric_Pad1.15x1.40mm_HandSolder, F.Cu at (193.3, 24.2)
- added R6: R103, Resistor_SMD:R_0805_2012Metric_Pad1.15x1.40mm_HandSolder, F.Cu at (199.1, 18.4)
- added R7: R102, Resistor_SMD:R_0805_2012Metric_Pad1.15x1.40mm_HandSolder, F.Cu at (130.4, 44.3)
- added R8: R220, Resistor_SMD:R_0805_2012Metric_Pad1.15x1.40mm_HandSolder, F.Cu at (126.7, 44.3)
- added R9: R220, Resistor_SMD:R_0805_2012Metric_Pad1.15x1.40mm_HandSolder, F.Cu at (172.6, 28.0)
- added REF**: MountingHole_3.2mm_M3_DIN965, MountingHole:MountingHole_3.2mm_M3_DIN965, F.Cu at (10.0, 10.0)
- added REF**: MountingHole_3.2mm_M3_DIN965, MountingHole:MountingHole_3.2mm_M3_DIN965, F.Cu at (90.0, 10.0)
- added REF**: MountingHole_3.2mm_M3_DIN965, MountingHole:MountingHole_3.2mm_M3_DIN965, F.Cu at (10.0, 90.0)
- added REF**: MountingHole_3.2mm_M3_DIN965, MountingHole:MountingHole_3.2mm_M3_DIN965, F.Cu at (90.0, 90.0)
- added U10: GSM_SMA, w_conn_rf:sma_straight_32k101-400l5, F.Cu at (138.1, 40.0)
- added U11: BT_SMA, w_conn_rf:sma_straight_32k101-400l5, F.Cu at (170.7, 19.3)
- added U12: USB_PCB, footprint-lib:usb-PCB, F.Cu at (150.3, 44.2)
- added U13: SMA, w_conn_rf:sma_straight_32k101-400l5, F.Cu at (146.6, 52.3)
- added U2: STM32L011K4Tx, Package_QFP:LQFP-32_7x7mm_P0.8mm, F.Cu at (186.3, 20.6)
- added U3: footprint-lib_nano-sim-card-holder, footprint-lib:nano-sim-card-holder, F.Cu at (151.9, 23.8)
- added U4: SMF05C, Package_TO_SOT_SMD:SOT-363_SC-70-6_Handsoldering, F.Cu at (169.3, 24.5)
- added U5: SIM800C, footprint-lib:LCC110P1570X1760X250-42N, F.Cu at (134.9, 25.8)
- added U7: LD3985M33R_SOT23, Package_TO_SOT_SMD:SOT-23-5, F.Cu at (152.3, 56.4)
- added U8: NEO-6M, RF_Module:ublox_NEO, F.Cu at (132.0, 56.8)
- added U9: 24AA32A, Package_TO_SOT_SMD:SOT-23-8_Handsoldering, F.Cu at (152.8, 52.7)
- C11: value 100n -> C22pf; footprint Capacitor_SMD:C_0603_1608Metric_Pad1.05x0.95mm_HandSolder -> Capacitor_SMD:C_0805_2012Metric_Pad1.15x1.40mm_HandSolder
- C12: value 4.3p -> C104; footprint Capacitor_SMD:C_0603_1608Metric_Pad1.05x0.95mm_HandSolder -> Capacitor_SMD:C_0805_2012Metric_Pad1.15x1.40mm_HandSolder
- C13: value 4.3p -> TC107,6V; footprint Capacitor_SMD:C_0603_1608Metric_Pad1.05x0.95mm_HandSolder -> Capacitor_Tantalum_SMD:CP_EIA-3216-12_Kemet-S_Pad1.58x1.35mm_HandSolder
- C22: value 10u -> C104; footprint Capacitor_SMD:CP_Elec_3x5.4 -> Capacitor_SMD:C_0603_1608Metric_Pad1.05x0.95mm_HandSolder
- C7: value 100n -> C104; footprint Capacitor_SMD:C_0603_1608Metric_Pad1.05x0.95mm_HandSolder -> Capacitor_SMD:C_0805_2012Metric_Pad1.15x1.40mm_HandSolder
- D1: value LED -> LED_Small; footprint LED_SMD:LED_0805_2012Metric_Pad1.15x1.40mm_HandSolder -> LED_SMD:LED_0805_2012Metric_Castellated
- D2, D3: value RED -> LED_Small; footprint LED_SMD:LED_0805_2012Metric_Pad1.15x1.40mm_HandSolder -> LED_SMD:LED_0805_2012Metric_Castellated
- J1: value Conn_01x04 -> PWR_CONN; footprint Connector_PinHeader_1.27mm:PinHeader_1x04_P1.27mm_Vertical -> Connector_PinHeader_2.54mm:PinHeader_1x04_P2.54mm_Vertical
- J2, J3, J6: footprint Connector_PinHeader_1.27mm:PinHeader_1x08_P1.27mm_Vertical -> Connector_PinHeader_2.54mm:PinHeader_1x08_P2.54mm_Vertical
- J4: value Conn_02x04_Row_Letter_First -> Conn_02x04_Odd_Even
- J7: value Conn_01x08 -> Jack-DC; footprint Connector_PinHeader_1.27mm:PinHeader_1x08_P1.27mm_Vertical -> footprint-lib:CUI-PJ-102A_dc-barrel-jack
- JP10, JP11, JP13: value Jumper -> Jumper_NC_Small
- JP6, JP8: footprint Jumper:SolderJumper-2_P1.3mm_Bridged_Pad1.0x1.5mm -> Jumper:SolderJumper-2_P1.3mm_Open_TrianglePad1.0x1.5mm
- R1: value 510 -> R102
- R2: value 510 -> R511
- R3: value R -> R102
- SW1: value SW_SPST -> SW_Push; footprint Button_Switch_THT:SW_PUSH_6mm_H4.3mm -> w_switch:PCB_PUSH
- U1: value STM32L011K4Tx -> AMS1117-3.3; footprint Package_QFP:LQFP-32_7x7mm_P0.8mm -> Package_TO_SOT_SMD:SOT-223-3_TabPin2
- U6: value AMS1117-1.8 -> MIC29302BU; footprint Package_TO_SOT_SMD:SOT-223-3_TabPin2 -> Package_TO_SOT_SMD:TO-263-5_TabPin3
- Y1: value 32.768K -> O32.768K; footprint Crystal:Crystal_HC49-4H_Vertical -> Crystal:Crystal_C38-LF_D3.0mm_L8.0mm_Vertical
- moved C13 128.5 mm to (177.0, 41.1)
- moved C22 128.5 mm to (178.3, 31.1)
- moved D1 128.5 mm to (173.5, 38.8)
- moved D2 128.5 mm to (184.0, 27.2)
- moved D3 128.5 mm to (177.3, 34.1)
- moved J2 128.5 mm to (164.3, 31.4)
- moved J3 128.5 mm to (170.2, 20.1)
- moved J5 128.5 mm to (155.2, 37.7)
- moved J7 128.5 mm to (154.9, 25.8)
- moved JP1 128.5 mm to (189.9, 29.4)
- moved JP10 128.5 mm to (184.2, 36.9)
- moved JP11 128.5 mm to (189.9, 32.0)
- moved JP4 128.5 mm to (180.9, 34.3)
- moved JP5 128.5 mm to (177.1, 39.0)
- moved JP6 128.5 mm to (180.4, 38.4)
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Connections:
- C11 pad 1: /NRST -> /SIM800C/SIMDATA
- C12 pad 1: Net-(C12-Pad1) -> GND
- C12 pad 2: GND -> /SIM800C/SIMVCC
- C13 pad 1: Net-(C13-Pad1) -> VDD_SIM800C
- C22 pad 1: +5V -> +3V3
- C7 pad 1: +3V3 -> AVDD
- J1 pad 1: +5V -> VIN
- J1 pad 3: (no net) -> VDD_STM32
- J2 pad 1: /PA0 -> /stm32/PA0
- J2 pad 2: /PA1 -> /stm32/PA1
- J2 pad 3: /PA2 -> /stm32/PA2
- J2 pad 4: /PA3 -> /stm32/PA3
- J2 pad 5: /PA4 -> /stm32/PA4
- J2 pad 6: /PA5 -> /stm32/PA5
- J2 pad 7: /PA6 -> /stm32/PA6
- J2 pad 8: /PA7 -> /stm32/PA7
- J3 pad 1: /PA8 -> /stm32/PA8
- J3 pad 2: /PA9 -> /stm32/PA9
- J3 pad 3: /PA10 -> /stm32/PA10
- J3 pad 4: /PA11 -> /stm32/PA11
- J3 pad 5: /PA12 -> /stm32/PA12
- J3 pad 6: (no net) -> /stm32/PC14
- J3 pad 7: (no net) -> /stm32/PC15
- J3 pad 8: /PA15 -> /stm32/PA15
- J4 pad 1: (no net) -> VDD
- J4 pad 2: (no net) -> VDD
- J4 pad 3: (no net) -> /stm32/PA14
- J4 pad 4: (no net) -> Net-(J4-Pad4)
- J4 pad 5: (no net) -> GND
- J4 pad 6: (no net) -> GND
- J4 pad 7: (no net) -> /stm32/PA13
- J4 pad 8: (no net) -> /stm32/NRST
- J5 pad 1: Net-(C25-Pad1) -> +3V3
- J5 pad 2: +3V3 -> VDD_STM32
- J6 pad 1: /PB0 -> /stm32/PB0
- J6 pad 2: /PB1 -> /stm32/PB1
- J6 pad 3: /PB3 -> /stm32/PB3
- J6 pad 4: /PB4 -> /stm32/PB4
- J6 pad 5: /PB5 -> /stm32/PB5
- J6 pad 6: /PB6 -> /stm32/PB6
- J6 pad 7: /PB7 -> /stm32/PB7
- J6 pad 8: (no net) -> Net-(J6-Pad8)
- J7 pad 2: +3V3 -> GND
- JP1 pad 1: /PB3 -> /stm32/PB3
- JP10 pad 1: +3V3 -> Net-(FB1-Pad1)
- JP10 pad 2: (no net) -> VDD_STM32
- JP11 pad 1: GND -> Net-(JP11-Pad1)
- JP11 pad 2: Net-(JP11-Pad2) -> GND
- JP13 pad 1: GND -> Net-(JP13-Pad1)
- JP13 pad 2: Net-(JP13-Pad2) -> GND
- JP2 pad 1: +5V -> VIN_STM32
- JP3 pad 1: +3V3 -> VDD_STM32
- JP4 pad 1: /BOOT0 -> Net-(JP17-Pad1)
- JP5 pad 1: Net-(C12-Pad1) -> Net-(C3-Pad1)
- JP5 pad 2: Net-(JP5-Pad2) -> Net-(JP4-Pad2)
- JP6 pad 1: /PC14 -> /stm32/PC14
- JP6 pad 2: Net-(JP5-Pad2) -> Net-(JP4-Pad2)
- JP7 pad 1: Net-(C13-Pad1) -> Net-(C4-Pad1)
- JP8 pad 1: /PC15 -> /stm32/PC15
- R1 pad 1: Net-(JP1-Pad2) -> +5V
- R1 pad 2: Net-(D1-Pad2) -> Net-(D12-Pad2)
- R2 pad 1: Net-(JP3-Pad2) -> Net-(JP1-Pad2)
- R2 pad 2: Net-(D3-Pad2) -> Net-(D1-Pad2)
- R3 pad 1: Net-(JP4-Pad2) -> Net-(JP2-Pad2)
- R3 pad 2: GND -> Net-(D2-Pad2)
- SW1 pad 1: GND -> /stm32/NRST
- SW1 pad 2: /NRST -> GND
- U1 pad 1: +3V3 -> GND
- U1 pad 2: Net-(JP5-Pad2) -> Net-(C2-Pad1)
- U1 pad 3: Net-(JP7-Pad2) -> VIN_STM32
- U6 pad 1: GND -> VIN_GSM
- U6 pad 2: Net-(C25-Pad1) -> VIN_GSM
- U6 pad 3: +5V -> GND
- Y1 pad 1: Net-(C12-Pad1) -> Net-(C3-Pad1)
- Y1 pad 2: Net-(C13-Pad1) -> Net-(C4-Pad1)
Routing:
- net (no net): vias 0 -> 3
