File: PCB/GSM-GPS-tryout.kicad_pcb (KiCad board)
At the start: 2 copper layers, 90 x 90 mm, 105 parts, among them J1 PWR_CONN, J10 Conn_01x05, J11 Conn_01x02, J15 Conn_01x04, J2 Conn_01x08, J3 Conn_01x08, J4 Conn_02x04_Odd_Even, J5 Conn_01x02, J6 Conn_01x08, J7 Jack-DC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

Commit message: updte
Parts:
- added C23: C106, Capacitor_SMD:C_0805_2012Metric_Pad1.15x1.40mm_HandSolder, F.Cu at (97.2, 48.8)
- added C24: C106, Capacitor_SMD:C_0805_2012Metric_Pad1.15x1.40mm_HandSolder, F.Cu at (93.4, 50.9)
- added D13: LED_ORANGE, LED_SMD:LED_0805_2012Metric_Castellated, F.Cu at (88.6, 52.5)
- added D14: VBUS_STATUS, LED_SMD:LED_0805_2012Metric_Pad1.15x1.40mm_HandSolder, F.Cu at (85.0, 57.4)
- added D15: MBR120, Diode_SMD:D_SOD-123F, F.Cu at (85.3, 55.2)
- added J12: Conn_01x02, Connector_PinHeader_2.54mm:PinHeader_1x02_P2.54mm_Vertical, F.Cu at (84.9, 49.7)
- added R21: R102, Resistor_SMD:R_0805_2012Metric_Pad1.15x1.40mm_HandSolder, F.Cu at (89.4, 56.4)
- added R22: R222, Resistor_SMD:R_0805_2012Metric_Pad1.15x1.40mm_HandSolder, F.Cu at (93.1, 52.8)
- added R23: R102, Resistor_SMD:R_0805_2012Metric_Pad1.15x1.40mm_HandSolder, F.Cu at (84.9, 59.4)
- added U14: MCP73831, Package_TO_SOT_SMD:SOT-23-5_HandSoldering, F.Cu at (89.1, 49.7)
- added U15: USB_PCB, footprint-lib:usb-PCB, F.Cu at (5.09, 36.2)
- D1: value LED_Small -> PB3
- D12: value 5V_STATUS -> VBAT_STATUS
- D2: value LED_Small -> VIN_STATUS
- D3: value LED_Small -> VDD_STATUS
- moved C2 162.4 mm to (38.8, 68.3)
- moved R5 158.3 mm to (42.3, 71.4)
- moved C4 158.2 mm to (49.3, 67.6)
- moved C1 158.2 mm to (44.6, 68.5)
- moved D4 155.0 mm to (34.6, 71.2)
- moved JP14 152.2 mm to (54.0, 63.3)
- moved D2 152.0 mm to (38.5, 71.2)
- moved FB1 149.8 mm to (60.6, 64.4)
- moved JP12 148.0 mm to (57.7, 61.2)
- moved U6 147.5 mm to (33.3, 38.8), turned to 0 degrees
- moved J3 146.4 mm to (26.8, 49.7)
- moved U3 146.2 mm to (15.0, 75.0), turned to 270 degrees
- moved D1 146.1 mm to (30.8, 70.2)
- moved JP11 145.8 mm to (49.1, 69.8)
- moved JP3 144.7 mm to (56.2, 68.8)
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Connections:
- J7 pad 1: +5V -> VBUS
- JP15 pad 1: +5V -> VBUS
- JP16 pad 1: +5V -> VBUS
- JP9 pad 1: +5V -> VBUS
- R1 pad 1: +5V -> VBAT
Routing:
- net (no net): vias 3 -> 0
Other:
- outline, holes or cut-outs redrawn

Commit message: updte
Parts:
- removed U12: USB_PCB, footprint-lib:usb-PCB
- added J13: SIM800_DEBUG, w_conn_pc:conn_usb_B_micro_smd, F.Cu at (22.5, 7.00)
- moved J3 56.9 mm to (75.0, 80.0), turned to 180 degrees
- moved U13 28.0 mm to (80.0, 10.0)
- moved U2 27.1 mm to (62.5, 77.5)
- moved U1 20.3 mm to (45.0, 82.5)
- moved C1 16.4 mm to (36.0, 82.5)
Changed lines of the file:
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@@
     (zones 0)
     (modules 116)
-    (nets 133)
+    (nets 134)
   )
   (page A4)
@@
   (net 131 "Net-(U15-Pad2)")
   (net 132 "Net-(U15-Pad3)")
+  (net 133 "Net-(J13-Pad4)")
   (net_class Default "This is the default net class."
     (clearance 0.2)
@@
     (add_net "Net-(D9-Pad2)")
     (add_net "Net-(FB1-Pad1)")
+    (add_net "Net-(J13-Pad4)")
     (add_net "Net-(J4-Pad4)")
     (add_net "Net-(J6-Pad8)")
@@
     (add_net VIN_STM32)
   )
+  (module w_conn_pc:conn_usb_B_micro_smd (layer F.Cu)
+    (at 22.53874 7 180)
+    (descr "USB B micro SMD connector, Molex P/N 47346-0001")
+    (fp_text reference J13 (at 0 2.60096 180) (layer F.SilkS)
+      (effects (font (size 0.50038 0.50038) (thickness 0.09906)))
+    )
+    (fp_text value SIM800_DEBUG (at 0 -4.0005 180) (layer F.SilkS)
+      (effects (font (size 0.50038 0.50038) (thickness 0.09906)))
+    )
+    (fp_line (start -4.20116 1.99898) (end 4.20116 1.99898) (layer F.SilkS) (width 0.20066))
+    (fp_line (start -4.20116 2.10058) (end 4.20116 2.10058) (layer F.SilkS) (width 0.20066))
+    (fp_line (start 4.20116 2.10058) (end 4.20116 1.89992) (layer F.SilkS) (width 0.20066))
+    (fp_line (start 4.20116 1.89992) (end -4.20116 1.89992) (layer F.SilkS) (width 0.20066))
+    (fp_line (start -4.20116 1.89992) (end -4.20116 2.10058) (layer F.SilkS) (width 0.20066))
+    (fp_line (start -3.8989 2.10058) (end -3.8989 -2.90068) (layer F.SilkS) (width 0.20066))
+    (fp_line (start -3.8989 -2.90068) (end 3.8989 -2.90068) (layer F.SilkS) (width 0.20066))
+    (fp_line (start 3.8989 -2.90068) (end 3.8989 2.10058) (layer F.SilkS) (width 0.20066))
+    (pad "" smd rect (at -0.8382 0 180) (size 1.17348 1.89738) (layers F.Cu F.Paste F.Mask))
+    (pad "" smd rect (at 0.8382 0 180) (size 1.17348 1.89738) (layers F.Cu F.Paste F.Mask))
+    (pad "" smd rect (at 2.91338 0 180) (size 2.3749 1.89738) (layers F.Cu F.Paste F.Mask))
+    (pad "" smd rect (at -2.91338 0 180) (size 2.3749 1.89738) (layers F.Cu F.Paste F.Mask))
+    (pad "" smd rect (at 2.46126 -2.2987 180) (size 1.4732 2.10058) (layers F.Cu F.Paste F.Mask))
+    (pad "" smd rect (at -2.46126 -2.2987 180) (size 1.4732 2.10058) (layers F.Cu F.Paste F.Mask))
+    (pad 1 smd rect (at -1.30048 -2.65938 180) (size 0.44958 1.37922) (layers F.Cu F.Paste F.Mask)
+      (net 20 /SIM800C/USB_VBUS))
+    (pad 2 smd rect (at -0.65024 -2.65938 180) (size 0.44958 1.37922) (layers F.Cu F.Paste F.Mask)
+      (net 18 /SIM800C/DP-))
+    (pad 3 smd rect (at 0 -2.65938 180) (size 0.44958 1.37922) (layers F.Cu F.Paste F.Mask)
+      (net 19 /SIM800C/DP+))
+    (pad 4 smd rect (at 0.65024 -2.65938 180) (size 0.44958 1.37922) (layers F.Cu F.Paste F.Mask)
+      (net 133 "Net-(J13-Pad4)"))
+    (pad 5 smd rect (at 1.30048 -2.65938 180) (size 0.44958 1.37922) (layers F.Cu F.Paste F.Mask)
+      (net 1 GND))
+    (model ${HOME}/_workspace/kicad/kicad_library/smisioto-footprints/modules/packages3d/walter/conn_pc/usb_B_micro_smd.wrl
+      (at (xyz 0 0 0))
+      (scale (xyz 1 1 1))
+      (rotate (xyz 0 0 0))
+    )
+  )
   (module Battery:BatteryHolder_Seiko_MS621F (layer F.Cu)
     (at 80 85 90)
@@
   )
   (module Capacitor_SMD:CP_Elec_3x5.4 (layer F.Cu)
-    (at 44.575001 68.535001)
+    (at 36 82.5)
     (descr "SMT capacitor, aluminium electrolytic, 3x5.4, Nichicon ")
     (tags "Capacitor Electrolytic")
@@
   )
   (module Connector_PinHeader_2.54mm:PinHeader_1x08_P2.54mm_Vertical (layer F.Cu)
-    (at 26.825001 49.685001)
+    (at 75 80 180)
     (descr "Through hole straight pin header, 1x08, 2.54mm pitch, single row")
     (tags "Through hole pin header THT 1x08 2.54mm single row")
-    (fp_text reference J3 (at 0 -2.33) (layer F.SilkS)
+    (fp_text reference J3 (at 0 -2.33 180) (layer F.SilkS)
       (effects (font (size 1 1) (thickness 0.15)))
     )
-    (fp_text value Conn_01x08 (at 0 20.11) (layer F.Fab)
+    (fp_text value Conn_01x08 (at 0 20.11 180) (layer F.Fab)
       (effects (font (size 1 1) (thickness 0.15)))
     )
@@
     (fp_line (start 1.8 19.55) (end 1.8 -1.8) (layer F.CrtYd) (width 0.05))
     (fp_line (start 1.8 -1.8) (end -1.8 -1.8) (layer F.CrtYd) (width 0.05))
-    (fp_text user %R (at 0 8.89 90) (layer F.Fab)
+    (fp_text user %R (at 0 8.89 270) (layer F.Fab)
       (effects (font (size 1 1) (thickness 0.15)))
     )
-    (pad 1 thru_hole rect (at 0 0) (size 1.7 1.7) (drill 1) (layers *.Cu *.Mask)
+    (pad 1 thru_hole rect (at 0 0 180) (size 1.7 1.7) (drill 1) (layers *.Cu *.Mask)
       (net 98 /stm32/PA8))
-    (pad 2 thru_hole oval (at 0 2.54) (size 1.7 1.7) (drill 1) (layers *.Cu *.Mask)
+    (pad 2 thru_hole oval (at 0 2.54 180) (size 1.7 1.7) (drill 1) (layers *.Cu *.Mask)
       (net 99 /stm32/PA9))
-    (pad 3 thru_hole oval (at 0 5.08) (size 1.7 1.7) (drill 1) (layers *.Cu *.Mask)
+    (pad 3 thru_hole oval (at 0 5.08 180) (size 1.7 1.7) (drill 1) (layers *.Cu *.Mask)
       (net 100 /stm32/PA10))
-    (pad 4 thru_hole oval (at 0 7.62) (size 1.7 1.7) (drill 1) (layers *.Cu *.Mask)
+    (pad 4 thru_hole oval (at 0 7.62 180) (size 1.7 1.7) (drill 1) (layers *.Cu *.Mask)
       (net 101 /stm32/PA11))
-    (pad 5 thru_hole oval (at 0 10.16) (size 1.7 1.7) (drill 1) (layers *.Cu *.Mask)
+    (pad 5 thru_hole oval (at 0 10.16 180) (size 1.7 1.7) (drill 1) (layers *.Cu *.Mask)
       (net 102 /stm32/PA12))
-    (pad 6 thru_hole oval (at 0 12.7) (size 1.7 1.7) (drill 1) (layers *.Cu *.Mask)
+    (pad 6 thru_hole oval (at 0 12.7 180) (size 1.7 1.7) (drill 1) (layers *.Cu *.Mask)
       (net 114 /stm32/PC14))
-    (pad 7 thru_hole oval (at 0 15.24) (size 1.7 1.7) (drill 1) (layers *.Cu *.Mask)
+    (pad 7 thru_hole oval (at 0 15.24 180) (size 1.7 1.7) (drill 1) (layers *.Cu *.Mask)
       (net 113 /stm32/PC15))
-    (pad 8 thru_hole oval (at 0 17.78) (size 1.7 1.7) (drill 1) (layers *.Cu *.Mask)
+    (pad 8 thru_hole oval (at 0 17.78 180) (size 1.7 1.7) (drill 1) (layers *.Cu *.Mask)
       (net 105 /stm32/PA15))
     (model ${KISYS3DMOD}/Connector_PinHeader_2.54mm.3dshapes/PinHeader_1x08_P2.54mm_Vertical.wrl
@@
   )
   (module Package_QFP:LQFP-32_7x7mm_P0.8mm (layer F.Cu)
-    (at 50.925001 52.985001)
+    (at 62.5 77.5)
     (descr "LQFP32: plastic low profile quad flat package; 32 leads; body 7 x 7 x 1.4 mm (see NXP sot358-1_po.pdf and sot358-1_fr.pdf)")
     (tags "QFP 0.8")
@@
   )
   (module Package_TO_SOT_SMD:SOT-223-3_TabPin2 (layer F.Cu)
-    (at 40.375001 62.735001)
+    (at 45 82.5)
     (descr "module CMS SOT223 4 pins")
     (tags "CMS SOT")
@@
       (net 25 "Net-(R9-Pad1)"))
   )
-  (module footprint-lib:usb-PCB (layer F.Cu)
-    (at 69.525001 24.575001)
-    (attr virtual)
-    (fp_text reference U12 (at 0.13 -7.85) (layer F.SilkS) hide
-      (effects (font (size 1.5 1.5) (thickness 0.15)))
-    )
-    (fp_text value USB_PCB (at 0.29 -10.13) (layer F.SilkS) hide
-      (effects (font (size 1.5 1.5) (thickness 0.15)))
-    )
-    (fp_line (start -6.03 0) (end -6.03 -12) (layer Dwgs.User) (width 0.15))
-    (fp_line (start 6.03 0) (end -6.03 0) (layer Dwgs.User) (width 0.15))
-    (fp_line (start 6.03 0) (end 6.03 -12) (layer Dwgs.User) (width 0.15))
-    (fp_text user VCC (at 3.81 -11.43 90) (layer F.SilkS)
-      (effects (font (size 1 1) (thickness 0.15)))
-    )
-    (fp_text user DP- (at 1.27 -11.43 90) (layer F.SilkS)
-      (effects (font (size 1 1) (thickness 0.15)))
-    )
-    (fp_text user DP+ (at -1.27 -11.43 90) (layer F.SilkS)
-      (effects (font (size 1 1) (thickness 0.15)))
-    )
-    (fp_text user GND (at -3.81 -11.43 90) (layer F.SilkS)
-      (effects (font (size 1 1) (thickness 0.15)))
-    )
-    (pad 2 connect rect (at 1.3 -5.15) (size 2 7.5) (layers F.Cu F.Mask)
-      (net 18 /SIM800C/DP-))
-    (pad 3 connect rect (at -1.3 -5.15) (size 2 7.5) (layers F.Cu F.Mask)
-      (net 19 /SIM800C/DP+))
-    (pad 4 connect rect (at -3.81 -4.9) (size 1.9 8) (layers F.Cu F.Mask)
-      (net 1 GND))
-    (pad 1 connect rect (at 3.81 -4.9) (size 1.9 8) (layers F.Cu F.Mask)
-      (net 20 /SIM800C/USB_VBUS))
-  )
   (module w_conn_rf:sma_straight_32k101-400l5 (layer F.Cu)
     (at 51.86 40.06)
@@
   )
   (module w_conn_rf:sma_straight_32k101-400l5 (layer F.Cu)
-    (at 107.33 16.29)
+    (at 80 10)
     (descr "SMA straight female connector, Rosenberger 32K101-400L5")
     (fp_text reference U13 (at 0 4.8) (layer F.SilkS)
