File: PCB/ublox-gps.sch (KiCad schematic (older format))
At the start: 17 parts, among them J15 Conn_01x04, J16 Conn_Coaxial, U7 LD3985M33R_SOT23, U8 NEO-6M, U9 24AA32A

Commit message: update
Parts:
- removed C17: 1u, Capacitor_SMD:C_0805_2012Metric_Pad1.15x1.40mm_HandSolder, symbol Device:C
- removed C18: 10u, Capacitor_SMD:C_0805_2012Metric_Pad1.15x1.40mm_HandSolder, symbol Device:C
- removed C19, C20: 0.1u, Capacitor_SMD:C_0805_2012Metric_Pad1.15x1.40mm_HandSolder, symbol Device:C
- removed D10, D9: LED, LED_SMD:LED_0805_2012Metric_Pad1.15x1.40mm_HandSolder, symbol Device:LED
- removed D11: 1N5817, Diode_THT:D_DO-41_SOD81_P10.16mm_Horizontal, symbol Diode:1N5817
- removed L1: 22u, Inductor_SMD:L_0805_2012Metric_Pad1.15x1.40mm_HandSolder, symbol Device:L
- removed R29, R31: 1k, Resistor_SMD:R_0805_2012Metric_Pad1.15x1.40mm_HandSolder, symbol Device:R
- removed R30: 22, Resistor_SMD:R_0805_2012Metric_Pad1.15x1.40mm_HandSolder, symbol Device:R
- added C?: C105, symbol taobao-c:C105
- added C?: C106, symbol taobao-c:C106
- added C? (x2): C104, symbol taobao-c:C104
- added D?: 1N5817, symbol Device:D_Zener_Small
- added D? (x2): LED_Small, symbol Device:LED_Small
- added L?: 22u, symbol Device:L_Small
- added R? (x2): R102, symbol taobao-r:R102
- added R?: R220, symbol taobao-r:R220
Changed lines of the file:
@@
-$EndComp
-$Comp
-L Device:R R29
-U 1 1 5BBAE2C3
-P 2700 4400
-F 0 "R29" V 2403 4400 50  0000 C CNN
-F 1 "1k" V 2494 4400 50  0000 C CNN
-F 2 "Resistor_SMD:R_0805_2012Metric_Pad1.15x1.40mm_HandSolder" V 2585 4400 50  0001 C CNN
-F 3 "~" H 2700 4400 50  0001 C CNN
-F 4 "0805" V 2585 4400 50  0000 C CNN "Field4"
-	1    2700 4400
-	0    1    1    0
-$EndComp
-$Comp
-L Device:LED D9
-U 1 1 5BBAE379
-P 2100 4400
-F 0 "D9" H 2091 4616 50  0000 C CNN
-F 1 "LED" H 2091 4525 50  0000 C CNN
-F 2 "LED_SMD:LED_0805_2012Metric_Pad1.15x1.40mm_HandSolder" H 2100 4400 50  0001 C CNN
-F 3 "~" H 2100 4400 50  0001 C CNN
-	1    2100 4400
-	1    0    0    -1
 $EndComp
 $Comp
@@
 $EndComp
 Wire Wire Line
-	2850 4400 3600 4400
-Wire Wire Line
-	2250 4400 2550 4400
-Wire Wire Line
 	1600 4400 1950 4400
 Text Label 3050 4400 0    50   ~ 0
@@
 Wire Wire Line
 	3300 5400 3300 5550
-$Comp
-L Device:L L1
-U 1 1 5BBAEB54
-P 2850 5000
-F 0 "L1" V 2750 5000 50  0000 C CNN
-F 1 "22u" V 2650 5000 50  0000 C CNN
-F 2 "Inductor_SMD:L_0805_2012Metric_Pad1.15x1.40mm_HandSolder" H 2850 5000 50  0001 C CNN
-F 3 "~" H 2850 5000 50  0001 C CNN
-F 4 "0805" V 2550 5000 50  0000 C CNN "Field4"
-	1    2850 5000
-	0    -1   -1   0
-$EndComp
 Wire Wire Line
 	2700 5000 2600 5000
@@
 Wire Wire Line
 	2600 5300 3600 5300
-$Comp
-L Device:R R30
-U 1 1 5BBAECA7
-P 3250 5000
-F 0 "R30" V 3043 5000 50  0000 C CNN
-F 1 "22" V 3134 5000 50  0000 C CNN
-F 2 "Resistor_SMD:R_0805_2012Metric_Pad1.15x1.40mm_HandSolder" V 3180 5000 50  0001 C CNN
-F 3 "~" H 3250 5000 50  0001 C CNN
-	1    3250 5000
-	0    1    1    0
-$EndComp
-Wire Wire Line
-	3000 5000 3100 5000
-Wire Wire Line
-	3400 5000 3500 5000
 $Comp
 L power:GND #PWR0162
@@
 	1    0    0    -1
 $EndComp
-$Comp
-L Diode:1N5817 D11
-U 1 1 5BBB0404
-P 6200 4050
-F 0 "D11" V 6246 3971 50  0000 R CNN
-F 1 "1N5817" V 6155 3971 50  0000 R CNN
-F 2 "Diode_THT:D_DO-41_SOD81_P10.16mm_Horizontal" H 6200 3875 50  0001 C CNN
-F 3 "http://www.vishay.com/docs/88525/1n5817.pdf" H 6200 4050 50  0001 C CNN
-	1    6200 4050
-	0    -1   -1   0
-$EndComp
-$Comp
-L Device:R R31
-U 1 1 5BBB0554
-P 6000 4400
-F 0 "R31" V 5793 4400 50  0000 C CNN
-F 1 "1k" V 5884 4400 50  0000 C CNN
-F 2 "Resistor_SMD:R_0805_2012Metric_Pad1.15x1.40mm_HandSolder" V 5930 4400 50  0001 C CNN
-F 3 "~" H 6000 4400 50  0001 C CNN
-	1    6000 4400
-	0    1    1    0
-$EndComp
 Wire Wire Line
 	5100 4400 5800 4400
 Wire Wire Line
 	6200 4200 6200 4400
-Wire Wire Line
-	6200 4400 6150 4400
-Wire Wire Line
-	6200 3800 6200 3900
 $Comp
 L Device:Battery BT1
@@
 	5800 4400 5800 4500
 Connection ~ 5800 4400
-Wire Wire Line
-	5800 4400 5850 4400
 $Comp
 L power:GND #PWR0165
@@
 	1    0    0    -1
 $EndComp
-$Comp
-L Device:C C17
-U 1 1 5BBBE031
-P 2000 1850
-F 0 "C17" H 2115 1941 50  0000 L CNN
-F 1 "1u" H 2115 1850 50  0000 L CNN
-F 2 "Capacitor_SMD:C_0805_2012Metric_Pad1.15x1.40mm_HandSolder" H 2038 1700 50  0001 C CNN
-F 3 "~" H 2000 1850 50  0001 C CNN
-F 4 "0805" H 2115 1759 50  0000 L CNN "Sch-footprint"
-	1    2000 1850
-	1    0    0    -1
-$EndComp
 Wire Wire Line
 	2000 1400 2000 1650
@@
 $EndComp
 Wire Wire Line
-	2000 2000 2000 2350
-Wire Wire Line
 	2450 1650 2300 1650
 Connection ~ 2000 1650
-Wire Wire Line
-	2000 1650 2000 1700
 Wire Wire Line
 	2450 1750 2300 1750
@@
 	2750 2350 2750 2050
 $Comp
-L Device:C C18
-U 1 1 5BBC3EC2
-P 3400 1850
-F 0 "C18" H 3515 1941 50  0000 L CNN
-F 1 "10u" H 3515 1850 50  0000 L CNN
-F 2 "Capacitor_SMD:C_0805_2012Metric_Pad1.15x1.40mm_HandSolder" H 3438 1700 50  0001 C CNN
-F 3 "~" H 3400 1850 50  0001 C CNN
-F 4 "0805" H 3515 1759 50  0000 L CNN "Sch-footprint"
-	1    3400 1850
-	1    0    0    -1
-$EndComp
-$Comp
-L Device:C C19
-U 1 1 5BBC3F04
-P 3800 1850
-F 0 "C19" H 3915 1941 50  0000 L CNN
-F 1 "0.1u" H 3915 1850 50  0000 L CNN
-F 2 "Capacitor_SMD:C_0805_2012Metric_Pad1.15x1.40mm_HandSolder" H 3838 1700 50  0001 C CNN
-F 3 "~" H 3800 1850 50  0001 C CNN
-F 4 "0805" H 3915 1759 50  0000 L CNN "Sch-footprint"
-	1    3800 1850
-	1    0    0    -1
-$EndComp
-$Comp
-L Device:C C20
-U 1 1 5BBC3F40
-P 4200 1850
-F 0 "C20" H 4315 1941 50  0000 L CNN
-F 1 "0.1u" H 4315 1850 50  0000 L CNN
-F 2 "Capacitor_SMD:C_0805_2012Metric_Pad1.15x1.40mm_HandSolder" H 4238 1700 50  0001 C CNN
-F 3 "~" H 4200 1850 50  0001 C CNN
-F 4 "0805" H 4315 1759 50  0000 L CNN "Sch-footprint"
-	1    4200 1850
-	1    0    0    -1
-$EndComp
-$Comp
 L customized_power:+3V3 #PWR0175
 U 1 1 5BBC4080
@@
 	3050 1650 3400 1650
 Connection ~ 4200 1650
-Wire Wire Line
-	4200 1650 4200 1700
-Wire Wire Line
-	3400 1650 3400 1700
 Connection ~ 3400 1650
 Wire Wire Line
 	3400 1650 3800 1650
-Wire Wire Line
-	3800 1650 3800 1700
 Connection ~ 3800 1650
 Wire Wire Line
@@
 $EndComp
 Wire Wire Line
-	3400 2000 3400 2150
-Wire Wire Line
 	3400 2150 3700 2150
-Wire Wire Line
-	4200 2150 4200 2000
-Wire Wire Line
-	3800 2000 3800 2150
 Connection ~ 3800 2150
 Wire Wire Line
@@
 Wire Wire Line
 	3700 2150 3800 2150
-$Comp
-L Device:LED D10
-U 1 1 5BBCC777
-P 4750 1900
-F 0 "D10" V 4788 1783 50  0000 R CNN
-F 1 "LED" V 4697 1783 50  0000 R CNN
-F 2 "LED_SMD:LED_0805_2012Metric_Pad1.15x1.40mm_HandSolder" H 4750 1900 50  0001 C CNN
-F 3 "~" H 4750 1900 50  0001 C CNN
-	1    4750 1900
-	0    -1   -1   0
-$EndComp
 $Comp
 L power:GND #PWR0177
@@
 	1    0    0    -1
 $EndComp
-Wire Wire Line
-	4750 2350 4750 2050
 Wire Wire Line
 	4200 1650 4750 1650
@@
 	2450 5300 2600 5300
 Connection ~ 2600 5300
+$Comp
+L taobao-r:R102 R?
+U 1 1 5BC45900
+P 6000 4400
+F 0 "R?" V 5750 4400 50  0000 C CNN
+F 1 "R102" V 5850 4400 50  0000 C CNN
+F 2 "" V 5930 4400 50  0001 C CNN
+F 3 "~" H 6000 4400 50  0001 C CNN
+	1    6000 4400
+	0    1    1    0
+$EndComp
+$Comp
+L taobao-r:R220 R?
+U 1 1 5BC45B9E
+P 3250 5000
+F 0 "R?" V 3000 5000 50  0000 C CNN
+F 1 "R220" V 3100 5000 50  0000 C CNN
+F 2 "" V 3180 5000 50  0001 C CNN
+F 3 "~" H 3250 5000 50  0001 C CNN
+	1    3250 5000
+	0    1    1    0
+$EndComp
+$Comp
+L taobao-r:R102 R?
+U 1 1 5BC46037
+P 2700 4400
+F 0 "R?" V 2450 4400 50  0000 C CNN
+F 1 "R102" V 2550 4400 50  0000 C CNN
+F 2 "" V 2630 4400 50  0001 C CNN
+F 3 "~" H 2700 4400 50  0001 C CNN
+	1    2700 4400
+	0    1    1    0
+$EndComp
+$Comp
+L taobao-c:C105 C?
+U 1 1 5BC4709A
+P 2000 1850
+F 0 "C?" H 2150 1900 50  0000 L CNN
+F 1 "C105" H 2150 1850 50  0000 L CNN
+F 2 "" H 2038 1700 50  0001 C CNN
+F 3 "~" H 2000 1850 50  0001 C CNN
+	1    2000 1850
+	1    0    0    -1
+$EndComp
+$Comp
+L taobao-c:C106 C?
+U 1 1 5BC47AA7
+P 3400 1850
+F 0 "C?" H 3550 1900 50  0000 L CNN
+F 1 "C106" H 3550 1850 50  0000 L CNN
+F 2 "" H 3438 1700 50  0001 C CNN
+F 3 "~" H 3400 1850 50  0001 C CNN
+	1    3400 1850
+	1    0    0    -1
+$EndComp
+$Comp
+L taobao-c:C104 C?
+U 1 1 5BC47C20
+P 3800 1850
+AR Path="/5BC47C20" Ref="C?"  Part="1"
+AR Path="/5BC0E426/5BC47C20" Ref="C?"  Part="1"
+F 0 "C?" H 3950 1900 50  0000 L CNN
+F 1 "C104" H 3950 1850 50  0000 L CNN
+F 2 "" H 3838 1700 50  0001 C CNN
+F 3 "~" H 3800 1850 50  0001 C CNN
+	1    3800 1850
+	1    0    0    -1
+$EndComp
+$Comp
+L taobao-c:C104 C?
+U 1 1 5BC47D54
+P 4200 1850
+AR Path="/5BC47D54" Ref="C?"  Part="1"
+AR Path="/5BC0E426/5BC47D54" Ref="C?"  Part="1"
+F 0 "C?" H 4350 1900 50  0000 L CNN
+F 1 "C104" H 4350 1850 50  0000 L CNN
+F 2 "" H 4238 1700 50  0001 C CNN
+F 3 "~" H 4200 1850 50  0001 C CNN
+	1    4200 1850
+	1    0    0    -1
+$EndComp
+Wire Wire Line
+	2000 1650 2000 1750
+Wire Wire Line
+	2000 1950 2000 2350
+Wire Wire Line
+	3400 1650 3400 1750
+Wire Wire Line
+	3400 1950 3400 2150
+Wire Wire Line
+	3800 1650 3800 1750
+Wire Wire Line
+	3800 1950 3800 2150
+Wire Wire Line
+	4200 1650 4200 1750
+Wire Wire Line
+	4200 1950 4200 2150
+Wire Wire Line
+	2800 4400 3600 4400
+Wire Wire Line
+	3350 5000 3500 5000
+Wire Wire Line
+	5800 4400 5900 4400
+Wire Wire Line
+	6100 4400 6200 4400
+$Comp
+L Device:D_Zener_Small D?
+U 1 1 5BD8793F
+P 6200 4100
+F 0 "D?" V 6250 4000 50  0000 R CNN
+F 1 "1N5817" V 6200 4000 50  0000 R CNN
+F 2 "" V 6200 4100 50  0001 C CNN
+F 3 "~" V 6200 4100 50  0001 C CNN
+	1    6200 4100
+	0    -1   -1   0
+$EndComp
+Wire Wire Line
+	6200 3800 6200 4000
+$Comp
+L Device:L_Small L?
+U 1 1 5BD89A25
+P 2800 5000
+F 0 "L?" V 3000 5000 50  0000 C CNN
+F 1 "22u" V 2900 5000 50  0000 C CNN
+F 2 "" H 2800 5000 50  0001 C CNN
+F 3 "~" H 2800 5000 50  0001 C CNN
+	1    2800 5000
+	0    -1   -1   0
+$EndComp
+Wire Wire Line
+	2900 5000 3150 5000
+$Comp
+L Device:LED_Small D?
+U 1 1 5BD8CAA6
+P 4750 1850
+F 0 "D?" V 4800 1750 50  0000 R CNN
+F 1 "LED_Small" V 4750 1750 50  0000 R CNN
+F 2 "" V 4750 1850 50  0001 C CNN
+F 3 "~" V 4750 1850 50  0001 C CNN
+	1    4750 1850
+	0    -1   -1   0
+$EndComp
+Wire Wire Line
+	4750 1950 4750 2350
+$Comp
+L Device:LED_Small D?
+U 1 1 5BD8ECDD
+P 2050 4400
+F 0 "D?" H 2050 4650 50  0000 C CNN
+F 1 "LED_Small" H 2050 4550 50  0000 C CNN
+F 2 "" V 2050 4400 50  0001 C CNN
+F 3 "~" V 2050 4400 50  0001 C CNN
+	1    2050 4400
+	1    0    0    -1
+$EndComp
+Wire Wire Line
+	2150 4400 2600 4400
 $EndSCHEMATC

Commit message: updte
Parts:
- removed D? (x2): LED_Small, symbol Device:LED_Small
- removed J16: Conn_Coaxial, Connector_Coaxial:U.FL_Hirose_U.FL-R-SMT-1_Vertical, symbol Connector:Conn_Coaxial
- added D?: LED_GREEN, symbol taobao-components:LED_RED
- added D?: LED_BLUE, symbol taobao-components:LED_BLUE
- added R?: R102, symbol taobao-r:R102
- added U?: SMA, w_conn_rf:sma_straight_32k101-400l5, symbol taobao-components:SMA
Connections:
- net +3V3: now also D?.2 (A)
- net GND: now also D?.1 (K), R?.2, U?.2 (GND)
- net GPS_ANT: now reaches L?.1, U8.11 (RF_IN)
- net GPS_ANT: now also U?.1 (RF)
- net at R?.2: now also D?.2 (A)
- new net: D?.1 (K), R?.1
Changed lines of the file:
@@
-$EndComp
-$Comp
-L Connector:Conn_Coaxial J16
-U 1 1 5BC108AE
-P 2250 5300
-F 0 "J16" H 2150 5550 50  0000 C CNN
-F 1 "Conn_Coaxial" H 2150 5500 50  0000 C CNN
-F 2 "Connector_Coaxial:U.FL_Hirose_U.FL-R-SMT-1_Vertical" H 2250 5300 50  0001 C CNN
-F 3 " ~" H 2250 5300 50  0001 C CNN
-	1    2250 5300
-	-1   0    0    -1
 $EndComp
 $Comp
 L power:GND #PWR0178
 U 1 1 5BC1AD1A
-P 2250 5550
-F 0 "#PWR0178" H 2250 5300 50  0001 C CNN
-F 1 "GND" H 2255 5377 50  0000 C CNN
-F 2 "" H 2250 5550 50  0001 C CNN
-F 3 "" H 2250 5550 50  0001 C CNN
-	1    2250 5550
-	1    0    0    -1
-$EndComp
-Wire Wire Line
-	2250 5500 2250 5550
-Wire Wire Line
-	2450 5300 2600 5300
+P 1400 5550
+F 0 "#PWR0178" H 1400 5300 50  0001 C CNN
+F 1 "GND" H 1405 5377 50  0000 C CNN
+F 2 "" H 1400 5550 50  0001 C CNN
+F 3 "" H 1400 5550 50  0001 C CNN
+	1    1400 5550
+	1    0    0    -1
+$EndComp
 Connection ~ 2600 5300
 $Comp
@@
 Wire Wire Line
 	2900 5000 3150 5000
-$Comp
-L Device:LED_Small D?
-U 1 1 5BD8CAA6
+Wire Wire Line
+	2150 4400 2600 4400
+$Comp
+L taobao-r:R102 R?
+U 1 1 5BCF2073
+P 4750 2150
+F 0 "R?" H 4809 2196 50  0000 L CNN
+F 1 "R102" H 4809 2105 50  0000 L CNN
+F 2 "" H 4750 2150 50  0001 C CNN
+F 3 "~" H 4750 2150 50  0001 C CNN
+	1    4750 2150
+	1    0    0    -1
+$EndComp
+$Comp
+L taobao-components:LED_RED D?
+U 1 1 5BCF2245
 P 4750 1850
-F 0 "D?" V 4800 1750 50  0000 R CNN
-F 1 "LED_Small" V 4750 1750 50  0000 R CNN
+F 0 "D?" V 4796 1782 50  0000 R CNN
+F 1 "LED_GREEN" V 4705 1782 50  0000 R CNN
 F 2 "" V 4750 1850 50  0001 C CNN
 F 3 "~" V 4750 1850 50  0001 C CNN
@@
 $EndComp
 Wire Wire Line
-	4750 1950 4750 2350
-$Comp
-L Device:LED_Small D?
-U 1 1 5BD8ECDD
+	4750 1950 4750 2050
+Wire Wire Line
+	4750 2250 4750 2350
+$Comp
+L taobao-components:LED_BLUE D?
+U 1 1 5BCF650D
 P 2050 4400
-F 0 "D?" H 2050 4650 50  0000 C CNN
-F 1 "LED_Small" H 2050 4550 50  0000 C CNN
+F 0 "D?" H 2050 4635 50  0000 C CNN
+F 1 "LED_BLUE" H 2050 4544 50  0000 C CNN
 F 2 "" V 2050 4400 50  0001 C CNN
 F 3 "~" V 2050 4400 50  0001 C CNN
@@
 	1    0    0    -1
 $EndComp
-Wire Wire Line
-	2150 4400 2600 4400
+$Comp
+L taobao-components:SMA U?
+U 1 1 5BCF65CE
+P 800 5350
+F 0 "U?" H 694 5715 50  0000 C CNN
+F 1 "SMA" H 694 5624 50  0000 C CNN
+F 2 "w_conn_rf:sma_straight_32k101-400l5" H 750 5300 50  0001 C CNN
+F 3 "" H 750 5300 50  0001 C CNN
+	1    800  5350
+	-1   0    0    -1
+$EndComp
+Text Label 2250 5300 0    50   ~ 0
+GPS_ANT
+Wire Wire Line
+	2250 5300 2600 5300
+Text Label 1600 5300 2    50   ~ 0
+GPS_ANT
+Wire Wire Line
+	1200 5300 1600 5300
+Wire Wire Line
+	1200 5450 1400 5450
+Wire Wire Line
+	1400 5450 1400 5550
+Text Label 1300 5450 0    50   ~ 0
+GPS_GND
+Text Label 3350 5200 0    50   ~ 0
+GPS_GND
 $EndSCHEMATC

Commit message: updte
Connections:
- net VCC renamed VIN_GPS
Other:
- moved on the sheet: J15
Changed lines of the file:
@@
 L Connector_Generic:Conn_01x04 J15
 U 1 1 5BBB2704
-P 7950 5550
-F 0 "J15" H 7870 5125 50  0000 C CNN
-F 1 "Conn_01x04" H 7870 5216 50  0000 C CNN
-F 2 "Connector_PinHeader_2.54mm:PinHeader_1x04_P2.54mm_Vertical" H 7950 5550 50  0001 C CNN
-F 3 "~" H 7950 5550 50  0001 C CNN
-	1    7950 5550
+P 900 1900
+F 0 "J15" H 820 1475 50  0000 C CNN
+F 1 "Conn_01x04" H 820 1566 50  0000 C CNN
+F 2 "Connector_PinHeader_2.54mm:PinHeader_1x04_P2.54mm_Vertical" H 900 1900 50  0001 C CNN
+F 3 "~" H 900 1900 50  0001 C CNN
+	1    900  1900
 	-1   0    0    1
 $EndComp
@@
 L power:GND #PWR0167
 U 1 1 5BBB2844
-P 8400 5800
-F 0 "#PWR0167" H 8400 5550 50  0001 C CNN
-F 1 "GND" H 8405 5627 50  0000 C CNN
-F 2 "" H 8400 5800 50  0001 C CNN
-F 3 "" H 8400 5800 50  0001 C CNN
-	1    8400 5800
-	1    0    0    -1
-$EndComp
-Wire Wire Line
-	8150 5650 8400 5650
-Wire Wire Line
-	8400 5650 8400 5800
-Text Label 8650 5450 2    50   ~ 0
+P 1350 2150
+F 0 "#PWR0167" H 1350 1900 50  0001 C CNN
+F 1 "GND" H 1355 1977 50  0000 C CNN
+F 2 "" H 1350 2150 50  0001 C CNN
+F 3 "" H 1350 2150 50  0001 C CNN
+	1    1350 2150
+	1    0    0    -1
+$EndComp
+Wire Wire Line
+	1100 2000 1350 2000
+Wire Wire Line
+	1350 2000 1350 2150
+Text Label 1600 1800 2    50   ~ 0
 RX
 Wire Wire Line
-	8650 5450 8150 5450
-Text Label 8650 5550 2    50   ~ 0
+	1600 1800 1100 1800
+Text Label 1600 1900 2    50   ~ 0
 TX
 Wire Wire Line
-	8650 5550 8150 5550
-Wire Wire Line
-	8400 5250 8400 5350
-Wire Wire Line
-	8400 5350 8150 5350
+	1600 1900 1100 1900
+Wire Wire Line
+	1350 1600 1350 1700
+Wire Wire Line
+	1350 1700 1100 1700
 $Comp
 L ublox:24AA32A U9
@@
 	1    0    0    -1
 $EndComp
-$Comp
-L customized_power:VCC #PWR0172
-U 1 1 5BBBDF82
-P 2000 1400
-F 0 "#PWR0172" H 2000 1250 50  0001 C CNN
-F 1 "VCC" H 2017 1573 50  0000 C CNN
-F 2 "" H 2000 1400 50  0001 C CNN
-F 3 "" H 2000 1400 50  0001 C CNN
-	1    2000 1400
-	1    0    0    -1
-$EndComp
 Wire Wire Line
 	2000 1400 2000 1650
@@
 NoConn ~ 3600 4600
 $Comp
-L customized_power:VCC #PWR0121
-U 1 1 5C0F17A2
-P 8400 5250
-F 0 "#PWR0121" H 8400 5100 50  0001 C CNN
-F 1 "VCC" H 8417 5423 50  0000 C CNN
-F 2 "" H 8400 5250 50  0001 C CNN
-F 3 "" H 8400 5250 50  0001 C CNN
-	1    8400 5250
-	1    0    0    -1
-$EndComp
-$Comp
 L power:GND #PWR0178
 U 1 1 5BC1AD1A
@@
 U 1 1 5BC45B9E
 P 3250 5000
-F 0 "R?" V 3000 5000 50  0000 C CNN
-F 1 "R220" V 3100 5000 50  0000 C CNN
+F 0 "R?" V 3054 5000 50  0000 C CNN
+F 1 "R220" V 3145 5000 50  0000 C CNN
 F 2 "" V 3180 5000 50  0001 C CNN
 F 3 "~" H 3250 5000 50  0001 C CNN
@@
 Text Label 3350 5200 0    50   ~ 0
 GPS_GND
+$Comp
+L taobao-components:VIN_GPS #PWR?
+U 1 1 5BD0DFE8
+P 2000 1400
+F 0 "#PWR?" H 2000 1250 50  0001 C CNN
+F 1 "VIN_GPS" H 2005 1523 50  0000 C CNN
+F 2 "" H 2000 1400 50  0001 C CNN
+F 3 "" H 2000 1400 50  0001 C CNN
+	1    2000 1400
+	1    0    0    -1
+$EndComp
+$Comp
+L taobao-components:VIN_GPS #PWR?
+U 1 1 5BD0E0E8
+P 1350 1600
+F 0 "#PWR?" H 1350 1450 50  0001 C CNN
+F 1 "VIN_GPS" H 1355 1723 50  0000 C CNN
+F 2 "" H 1350 1600 50  0001 C CNN
+F 3 "" H 1350 1600 50  0001 C CNN
+	1    1350 1600
+	1    0    0    -1
+$EndComp
 $EndSCHEMATC

Commit message: updte
Parts:
- removed D?: 1N5817, symbol Device:D_Zener_Small
- added D11: SD_1N5817_SS12, Diode_SMD:D_1206_3216Metric_Pad1.42x1.75mm_HandSolder, symbol taobao-sd:SD_1N5817_SS12
- C19, C20, C21, C22: renamed from C?; footprint (none) -> Capacitor_SMD:C_0603_1608Metric_Pad1.05x0.95mm_HandSolder
- D10, D9: renamed from D?; footprint (none) -> LED_SMD:LED_0805_2012Metric_Castellated
- L2: renamed from L?; footprint (none) -> w_smd_inductors:inductor_smd_0805
- R17, R18, R19, R20: renamed from R?; footprint (none) -> Resistor_SMD:R_0805_2012Metric_Pad1.15x1.40mm_HandSolder
- gave numbers to parts that had none: 1
Connections:
- net +3V3: now also D11.2 (A)
- net at R20.1: now also D11.1 (K)
Changed lines of the file:
@@
 Connection ~ 2600 5300
 $Comp
-L taobao-r:R102 R?
+L taobao-r:R102 R20
 U 1 1 5BC45900
 P 6000 4400
-F 0 "R?" V 5750 4400 50  0000 C CNN
+F 0 "R20" V 5750 4400 50  0000 C CNN
 F 1 "R102" V 5850 4400 50  0000 C CNN
-F 2 "" V 5930 4400 50  0001 C CNN
+F 2 "Resistor_SMD:R_0805_2012Metric_Pad1.15x1.40mm_HandSolder" V 5930 4400 50  0001 C CNN
 F 3 "~" H 6000 4400 50  0001 C CNN
 	1    6000 4400
@@
 $EndComp
 $Comp
-L taobao-r:R220 R?
+L taobao-r:R220 R18
 U 1 1 5BC45B9E
 P 3250 5000
-F 0 "R?" V 3054 5000 50  0000 C CNN
+F 0 "R18" V 3054 5000 50  0000 C CNN
 F 1 "R220" V 3145 5000 50  0000 C CNN
-F 2 "" V 3180 5000 50  0001 C CNN
+F 2 "Resistor_SMD:R_0805_2012Metric_Pad1.15x1.40mm_HandSolder" V 3180 5000 50  0001 C CNN
 F 3 "~" H 3250 5000 50  0001 C CNN
 	1    3250 5000
@@
 $EndComp
 $Comp
-L taobao-r:R102 R?
+L taobao-r:R102 R17
 U 1 1 5BC46037
 P 2700 4400
-F 0 "R?" V 2450 4400 50  0000 C CNN
+F 0 "R17" V 2450 4400 50  0000 C CNN
 F 1 "R102" V 2550 4400 50  0000 C CNN
-F 2 "" V 2630 4400 50  0001 C CNN
+F 2 "Resistor_SMD:R_0805_2012Metric_Pad1.15x1.40mm_HandSolder" V 2630 4400 50  0001 C CNN
 F 3 "~" H 2700 4400 50  0001 C CNN
 	1    2700 4400
@@
 $EndComp
 $Comp
-L taobao-c:C105 C?
+L taobao-c:C105 C19
 U 1 1 5BC4709A
 P 2000 1850
-F 0 "C?" H 2150 1900 50  0000 L CNN
+F 0 "C19" H 2150 1900 50  0000 L CNN
 F 1 "C105" H 2150 1850 50  0000 L CNN
-F 2 "" H 2038 1700 50  0001 C CNN
+F 2 "Capacitor_SMD:C_0603_1608Metric_Pad1.05x0.95mm_HandSolder" H 2038 1700 50  0001 C CNN
 F 3 "~" H 2000 1850 50  0001 C CNN
 	1    2000 1850
@@
 $EndComp
 $Comp
-L taobao-c:C106 C?
+L taobao-c:C106 C20
 U 1 1 5BC47AA7
 P 3400 1850
-F 0 "C?" H 3550 1900 50  0000 L CNN
+F 0 "C20" H 3550 1900 50  0000 L CNN
 F 1 "C106" H 3550 1850 50  0000 L CNN
-F 2 "" H 3438 1700 50  0001 C CNN
+F 2 "Capacitor_SMD:C_0603_1608Metric_Pad1.05x0.95mm_HandSolder" H 3438 1700 50  0001 C CNN
 F 3 "~" H 3400 1850 50  0001 C CNN
 	1    3400 1850
@@
 P 3800 1850
 AR Path="/5BC47C20" Ref="C?"  Part="1"
-AR Path="/5BC0E426/5BC47C20" Ref="C?"  Part="1"
-F 0 "C?" H 3950 1900 50  0000 L CNN
+AR Path="/5BC0E426/5BC47C20" Ref="C21"  Part="1"
+F 0 "C21" H 3950 1900 50  0000 L CNN
 F 1 "C104" H 3950 1850 50  0000 L CNN
-F 2 "" H 3838 1700 50  0001 C CNN
+F 2 "Capacitor_SMD:C_0603_1608Metric_Pad1.05x0.95mm_HandSolder" H 3838 1700 50  0001 C CNN
 F 3 "~" H 3800 1850 50  0001 C CNN
 	1    3800 1850
@@
 P 4200 1850
 AR Path="/5BC47D54" Ref="C?"  Part="1"
-AR Path="/5BC0E426/5BC47D54" Ref="C?"  Part="1"
-F 0 "C?" H 4350 1900 50  0000 L CNN
+AR Path="/5BC0E426/5BC47D54" Ref="C22"  Part="1"
+F 0 "C22" H 4350 1900 50  0000 L CNN
 F 1 "C104" H 4350 1850 50  0000 L CNN
-F 2 "" H 4238 1700 50  0001 C CNN
+F 2 "Capacitor_SMD:C_0603_1608Metric_Pad1.05x0.95mm_HandSolder" H 4238 1700 50  0001 C CNN
 F 3 "~" H 4200 1850 50  0001 C CNN
 	1    4200 1850
@@
 Wire Wire Line
 	6100 4400 6200 4400
-$Comp
-L Device:D_Zener_Small D?
-U 1 1 5BD8793F
-P 6200 4100
-F 0 "D?" V 6250 4000 50  0000 R CNN
-F 1 "1N5817" V 6200 4000 50  0000 R CNN
-F 2 "" V 6200 4100 50  0001 C CNN
-F 3 "~" V 6200 4100 50  0001 C CNN
-	1    6200 4100
-	0    -1   -1   0
-$EndComp
 Wire Wire Line
 	6200 3800 6200 4000
 $Comp
-L Device:L_Small L?
+L Device:L_Small L2
 U 1 1 5BD89A25
 P 2800 5000
-F 0 "L?" V 3000 5000 50  0000 C CNN
+F 0 "L2" V 3000 5000 50  0000 C CNN
 F 1 "22u" V 2900 5000 50  0000 C CNN
-F 2 "" H 2800 5000 50  0001 C CNN
+F 2 "w_smd_inductors:inductor_smd_0805" H 2800 5000 50  0001 C CNN
 F 3 "~" H 2800 5000 50  0001 C CNN
 	1    2800 5000
@@
 	2150 4400 2600 4400
 $Comp
-L taobao-r:R102 R?
+L taobao-r:R102 R19
 U 1 1 5BCF2073
 P 4750 2150
-F 0 "R?" H 4809 2196 50  0000 L CNN
+F 0 "R19" H 4809 2196 50  0000 L CNN
 F 1 "R102" H 4809 2105 50  0000 L CNN
-F 2 "" H 4750 2150 50  0001 C CNN
+F 2 "Resistor_SMD:R_0805_2012Metric_Pad1.15x1.40mm_HandSolder" H 4750 2150 50  0001 C CNN
 F 3 "~" H 4750 2150 50  0001 C CNN
 	1    4750 2150
@@
 $EndComp
 $Comp
-L taobao-components:LED_RED D?
+L taobao-components:LED_RED D10
 U 1 1 5BCF2245
 P 4750 1850
-F 0 "D?" V 4796 1782 50  0000 R CNN
+F 0 "D10" V 4796 1782 50  0000 R CNN
 F 1 "LED_GREEN" V 4705 1782 50  0000 R CNN
-F 2 "" V 4750 1850 50  0001 C CNN
+F 2 "LED_SMD:LED_0805_2012Metric_Castellated" V 4750 1850 50  0001 C CNN
 F 3 "~" V 4750 1850 50  0001 C CNN
 	1    4750 1850
@@
 	4750 2250 4750 2350
 $Comp
-L taobao-components:LED_BLUE D?
+L taobao-components:LED_BLUE D9
 U 1 1 5BCF650D
 P 2050 4400
-F 0 "D?" H 2050 4635 50  0000 C CNN
+F 0 "D9" H 2050 4635 50  0000 C CNN
 F 1 "LED_BLUE" H 2050 4544 50  0000 C CNN
-F 2 "" V 2050 4400 50  0001 C CNN
+F 2 "LED_SMD:LED_0805_2012Metric_Castellated" V 2050 4400 50  0001 C CNN
 F 3 "~" V 2050 4400 50  0001 C CNN
 	1    2050 4400
@@
 $EndComp
 $Comp
-L taobao-components:SMA U?
+L taobao-components:SMA U13
 U 1 1 5BCF65CE
 P 800 5350
-F 0 "U?" H 694 5715 50  0000 C CNN
+F 0 "U13" H 694 5715 50  0000 C CNN
 F 1 "SMA" H 694 5624 50  0000 C CNN
 F 2 "w_conn_rf:sma_straight_32k101-400l5" H 750 5300 50  0001 C CNN
@@
 	1    0    0    -1
 $EndComp
+$Comp
+L taobao-sd:SD_1N5817_SS12 D11
+U 1 1 5BE402D8
+P 6200 4100
+F 0 "D11" V 6246 4032 50  0000 R CNN
+F 1 "SD_1N5817_SS12" V 6155 4032 50  0000 R CNN
+F 2 "Diode_SMD:D_1206_3216Metric_Pad1.42x1.75mm_HandSolder" V 6200 4100 50  0001 C CNN
+F 3 "~" V 6200 4100 50  0001 C CNN
+	1    6200 4100
+	0    -1   -1   0
+$EndComp
 $EndSCHEMATC
