File: PCB/GSM-GPS-tryout.sch (KiCad schematic (older format))
At the start: 0 parts

Commit message: update
Parts:
- added D12: 5V_STATUS, LED_SMD:LED_0805_2012Metric_Pad1.15x1.40mm_HandSolder, symbol Device:LED
- added D13: 3V3_STATUS, LED_SMD:LED_0805_2012Metric_Pad1.15x1.40mm_HandSolder, symbol Device:LED
- added R32: 511, Resistor_SMD:R_0805_2012Metric_Pad1.15x1.40mm_HandSolder, symbol Device:R
- added R4: 102, Resistor_SMD:R_0805_2012Metric_Pad1.15x1.40mm_HandSolder, symbol Device:R
Connections:
- net labels added: +5V, 3V3, GND
- wire segments 0 -> 6
Changed lines of the file:
@@
 EELAYER 26 0
 EELAYER END
-$Descr A3 16535 11693
+$Descr A4 11693 8268
 encoding utf-8
 Sheet 1 4
@@
 $EndDescr
 $Sheet
-S 1150 850  1350 950
+S 1000 1050 1350 950
 U 5BB772CE
 F0 "stm32" 50
@@
 $EndSheet
 $Sheet
-S 2700 850  1400 950
+S 2550 1050 1400 950
 U 5BB83F82
 F0 "SIM800C" 50
@@
 $EndSheet
 $Sheet
-S 1000 2350 1250 950
+S 4300 1050 1250 950
 U 5BC0E426
 F0 "ublox-gps" 50
 F1 "ublox-gps.sch" 50
 $EndSheet
+$Comp
+L tinkerforge:3V3 #PWR0102
+U 1 1 5BC31334
+P 1950 2850
+F 0 "#PWR0102" H 1950 2700 50  0001 C CNN
+F 1 "3V3" H 1965 3023 50  0000 C CNN
+F 2 "" H 1950 2850 50  0000 C CNN
+F 3 "" H 1950 2850 50  0000 C CNN
+	1    1950 2850
+	1    0    0    -1
+$EndComp
+$Comp
+L Device:R R32
+U 1 1 5BC3136B
+P 1950 3200
+F 0 "R32" H 2020 3246 50  0000 L CNN
+F 1 "511" H 2020 3155 50  0000 L CNN
+F 2 "Resistor_SMD:R_0805_2012Metric_Pad1.15x1.40mm_HandSolder" V 1880 3200 50  0001 C CNN
+F 3 "~" H 1950 3200 50  0001 C CNN
+	1    1950 3200
+	1    0    0    -1
+$EndComp
+$Comp
+L Device:LED D13
+U 1 1 5BC313EB
+P 1950 3700
+F 0 "D13" V 1988 3582 50  0000 R CNN
+F 1 "3V3_STATUS" V 1897 3582 50  0000 R CNN
+F 2 "LED_SMD:LED_0805_2012Metric_Pad1.15x1.40mm_HandSolder" H 1950 3700 50  0001 C CNN
+F 3 "~" H 1950 3700 50  0001 C CNN
+	1    1950 3700
+	0    -1   -1   0
+$EndComp
+$Comp
+L power:GND #PWR0103
+U 1 1 5BC3147B
+P 1950 4000
+F 0 "#PWR0103" H 1950 3750 50  0001 C CNN
+F 1 "GND" H 1955 3827 50  0000 C CNN
+F 2 "" H 1950 4000 50  0001 C CNN
+F 3 "" H 1950 4000 50  0001 C CNN
+	1    1950 4000
+	1    0    0    -1
+$EndComp
+Wire Wire Line
+	1950 2850 1950 3050
+Wire Wire Line
+	1950 3350 1950 3550
+Wire Wire Line
+	1950 3850 1950 4000
+$Comp
+L Device:R R4
+U 1 1 5BC31525
+P 1450 3200
+F 0 "R4" H 1520 3246 50  0000 L CNN
+F 1 "102" H 1520 3155 50  0000 L CNN
+F 2 "Resistor_SMD:R_0805_2012Metric_Pad1.15x1.40mm_HandSolder" V 1380 3200 50  0001 C CNN
+F 3 "~" H 1450 3200 50  0001 C CNN
+	1    1450 3200
+	1    0    0    -1
+$EndComp
+$Comp
+L Device:LED D12
+U 1 1 5BC3152B
+P 1450 3700
+F 0 "D12" V 1488 3582 50  0000 R CNN
+F 1 "5V_STATUS" V 1397 3582 50  0000 R CNN
+F 2 "LED_SMD:LED_0805_2012Metric_Pad1.15x1.40mm_HandSolder" H 1450 3700 50  0001 C CNN
+F 3 "~" H 1450 3700 50  0001 C CNN
+	1    1450 3700
+	0    -1   -1   0
+$EndComp
+$Comp
+L power:GND #PWR0110
+U 1 1 5BC31531
+P 1450 4000
+F 0 "#PWR0110" H 1450 3750 50  0001 C CNN
+F 1 "GND" H 1455 3827 50  0000 C CNN
+F 2 "" H 1450 4000 50  0001 C CNN
+F 3 "" H 1450 4000 50  0001 C CNN
+	1    1450 4000
+	1    0    0    -1
+$EndComp
+Wire Wire Line
+	1450 2850 1450 3050
+Wire Wire Line
+	1450 3350 1450 3550
+Wire Wire Line
+	1450 3850 1450 4000
+$Comp
+L tinkerforge:+5V #PWR0111
+U 1 1 5BC3168D
+P 1450 2850
+F 0 "#PWR0111" H 1450 2700 50  0001 C CNN
+F 1 "+5V" H 1465 3023 50  0000 C CNN
+F 2 "" H 1450 2850 50  0000 C CNN
+F 3 "" H 1450 2850 50  0000 C CNN
+	1    1450 2850
+	1    0    0    -1
+$EndComp
 $EndSCHEMATC

Commit message: update
Parts:
- removed R32: 511, Resistor_SMD:R_0805_2012Metric_Pad1.15x1.40mm_HandSolder, symbol Device:R
- removed R4: 102, Resistor_SMD:R_0805_2012Metric_Pad1.15x1.40mm_HandSolder, symbol Device:R
- added R?: R511, symbol taobao-r:R511
- added R?: R102, symbol taobao-r:R102
Connections:
- net labels added: +3V3
- net labels removed: 3V3
Changed lines of the file:
@@
 $EndSheet
-$Comp
-L tinkerforge:3V3 #PWR0102
-U 1 1 5BC31334
-P 1950 2850
-F 0 "#PWR0102" H 1950 2700 50  0001 C CNN
-F 1 "3V3" H 1965 3023 50  0000 C CNN
-F 2 "" H 1950 2850 50  0000 C CNN
-F 3 "" H 1950 2850 50  0000 C CNN
-	1    1950 2850
-	1    0    0    -1
-$EndComp
-$Comp
-L Device:R R32
-U 1 1 5BC3136B
-P 1950 3200
-F 0 "R32" H 2020 3246 50  0000 L CNN
-F 1 "511" H 2020 3155 50  0000 L CNN
-F 2 "Resistor_SMD:R_0805_2012Metric_Pad1.15x1.40mm_HandSolder" V 1880 3200 50  0001 C CNN
-F 3 "~" H 1950 3200 50  0001 C CNN
-	1    1950 3200
-	1    0    0    -1
-$EndComp
 $Comp
 L Device:LED D13
@@
 $EndComp
 Wire Wire Line
-	1950 2850 1950 3050
-Wire Wire Line
-	1950 3350 1950 3550
-Wire Wire Line
 	1950 3850 1950 4000
-$Comp
-L Device:R R4
-U 1 1 5BC31525
-P 1450 3200
-F 0 "R4" H 1520 3246 50  0000 L CNN
-F 1 "102" H 1520 3155 50  0000 L CNN
-F 2 "Resistor_SMD:R_0805_2012Metric_Pad1.15x1.40mm_HandSolder" V 1380 3200 50  0001 C CNN
-F 3 "~" H 1450 3200 50  0001 C CNN
-	1    1450 3200
-	1    0    0    -1
-$EndComp
 $Comp
 L Device:LED D12
@@
 $EndComp
 Wire Wire Line
-	1450 2850 1450 3050
-Wire Wire Line
-	1450 3350 1450 3550
-Wire Wire Line
 	1450 3850 1450 4000
 $Comp
-L tinkerforge:+5V #PWR0111
-U 1 1 5BC3168D
+L power:+5V #PWR?
+U 1 1 5BC354AB
 P 1450 2850
-F 0 "#PWR0111" H 1450 2700 50  0001 C CNN
-F 1 "+5V" H 1465 3023 50  0000 C CNN
-F 2 "" H 1450 2850 50  0000 C CNN
-F 3 "" H 1450 2850 50  0000 C CNN
+F 0 "#PWR?" H 1450 2700 50  0001 C CNN
+F 1 "+5V" H 1500 3050 50  0000 C CNN
+F 2 "" H 1450 2850 50  0001 C CNN
+F 3 "" H 1450 2850 50  0001 C CNN
 	1    1450 2850
 	1    0    0    -1
 $EndComp
+$Comp
+L power:+3V3 #PWR?
+U 1 1 5BC35548
+P 1950 2850
+F 0 "#PWR?" H 1950 2700 50  0001 C CNN
+F 1 "+3V3" H 2000 3050 50  0000 C CNN
+F 2 "" H 1950 2850 50  0001 C CNN
+F 3 "" H 1950 2850 50  0001 C CNN
+	1    1950 2850
+	1    0    0    -1
+$EndComp
+$Comp
+L taobao-r:R511 R?
+U 1 1 5BC25737
+P 1950 3200
+F 0 "R?" H 2050 3250 50  0000 L CNN
+F 1 "R511" H 2050 3200 50  0000 L CNN
+F 2 "" H 1950 3200 50  0001 C CNN
+F 3 "~" H 1950 3200 50  0001 C CNN
+	1    1950 3200
+	1    0    0    -1
+$EndComp
+Wire Wire Line
+	1950 2850 1950 3100
+Wire Wire Line
+	1950 3300 1950 3550
+$Comp
+L taobao-r:R102 R?
+U 1 1 5BC258E4
+P 1450 3200
+F 0 "R?" H 1550 3250 50  0000 L CNN
+F 1 "R102" H 1550 3200 50  0000 L CNN
+F 2 "" H 1450 3200 50  0001 C CNN
+F 3 "~" H 1450 3200 50  0001 C CNN
+	1    1450 3200
+	1    0    0    -1
+$EndComp
+Wire Wire Line
+	1450 2850 1450 3100
+Wire Wire Line
+	1450 3300 1450 3550
 $EndSCHEMATC

Commit message: updte
Parts:
- removed D13: 3V3_STATUS, LED_SMD:LED_0805_2012Metric_Pad1.15x1.40mm_HandSolder, symbol Device:LED
- removed R?: R511, symbol taobao-r:R511
- added J?: Jack-DC, symbol Connector:Jack-DC
- added JP? (x3): Jumper_NO_Small, symbol Device:Jumper_NO_Small
Connections:
- net labels added: VIN_GPS, VIN_GSM, VIN_STM32
- net labels removed: +3V3
- wire segments 6 -> 17
Other:
- moved on the sheet: D12, R?
Changed lines of the file:
@@
 $EndSheet
-$Comp
-L Device:LED D13
-U 1 1 5BC313EB
-P 1950 3700
-F 0 "D13" V 1988 3582 50  0000 R CNN
-F 1 "3V3_STATUS" V 1897 3582 50  0000 R CNN
-F 2 "LED_SMD:LED_0805_2012Metric_Pad1.15x1.40mm_HandSolder" H 1950 3700 50  0001 C CNN
-F 3 "~" H 1950 3700 50  0001 C CNN
-	1    1950 3700
-	0    -1   -1   0
-$EndComp
-$Comp
-L power:GND #PWR0103
-U 1 1 5BC3147B
-P 1950 4000
-F 0 "#PWR0103" H 1950 3750 50  0001 C CNN
-F 1 "GND" H 1955 3827 50  0000 C CNN
-F 2 "" H 1950 4000 50  0001 C CNN
-F 3 "" H 1950 4000 50  0001 C CNN
-	1    1950 4000
-	1    0    0    -1
-$EndComp
-Wire Wire Line
-	1950 3850 1950 4000
 $Comp
 L Device:LED D12
 U 1 1 5BC3152B
-P 1450 3700
-F 0 "D12" V 1488 3582 50  0000 R CNN
-F 1 "5V_STATUS" V 1397 3582 50  0000 R CNN
-F 2 "LED_SMD:LED_0805_2012Metric_Pad1.15x1.40mm_HandSolder" H 1450 3700 50  0001 C CNN
-F 3 "~" H 1450 3700 50  0001 C CNN
-	1    1450 3700
+P 1000 4650
+F 0 "D12" V 1038 4532 50  0000 R CNN
+F 1 "5V_STATUS" V 947 4532 50  0000 R CNN
+F 2 "LED_SMD:LED_0805_2012Metric_Pad1.15x1.40mm_HandSolder" H 1000 4650 50  0001 C CNN
+F 3 "~" H 1000 4650 50  0001 C CNN
+	1    1000 4650
 	0    -1   -1   0
 $EndComp
@@
 L power:GND #PWR0110
 U 1 1 5BC31531
-P 1450 4000
-F 0 "#PWR0110" H 1450 3750 50  0001 C CNN
-F 1 "GND" H 1455 3827 50  0000 C CNN
-F 2 "" H 1450 4000 50  0001 C CNN
-F 3 "" H 1450 4000 50  0001 C CNN
-	1    1450 4000
+P 1000 4950
+F 0 "#PWR0110" H 1000 4700 50  0001 C CNN
+F 1 "GND" H 1005 4777 50  0000 C CNN
+F 2 "" H 1000 4950 50  0001 C CNN
+F 3 "" H 1000 4950 50  0001 C CNN
+	1    1000 4950
 	1    0    0    -1
 $EndComp
 Wire Wire Line
-	1450 3850 1450 4000
+	1000 4800 1000 4950
 $Comp
 L power:+5V #PWR?
 U 1 1 5BC354AB
-P 1450 2850
-F 0 "#PWR?" H 1450 2700 50  0001 C CNN
-F 1 "+5V" H 1500 3050 50  0000 C CNN
-F 2 "" H 1450 2850 50  0001 C CNN
-F 3 "" H 1450 2850 50  0001 C CNN
-	1    1450 2850
+P 1000 3800
+F 0 "#PWR?" H 1000 3650 50  0001 C CNN
+F 1 "+5V" H 1050 4000 50  0000 C CNN
+F 2 "" H 1000 3800 50  0001 C CNN
+F 3 "" H 1000 3800 50  0001 C CNN
+	1    1000 3800
 	1    0    0    -1
 $EndComp
 $Comp
-L power:+3V3 #PWR?
-U 1 1 5BC35548
-P 1950 2850
-F 0 "#PWR?" H 1950 2700 50  0001 C CNN
-F 1 "+3V3" H 2000 3050 50  0000 C CNN
-F 2 "" H 1950 2850 50  0001 C CNN
-F 3 "" H 1950 2850 50  0001 C CNN
-	1    1950 2850
+L taobao-r:R102 R?
+U 1 1 5BC258E4
+P 1000 4150
+F 0 "R?" H 1100 4200 50  0000 L CNN
+F 1 "R102" H 1100 4150 50  0000 L CNN
+F 2 "" H 1000 4150 50  0001 C CNN
+F 3 "~" H 1000 4150 50  0001 C CNN
+	1    1000 4150
+	1    0    0    -1
+$EndComp
+Wire Wire Line
+	1000 3800 1000 4050
+Wire Wire Line
+	1000 4250 1000 4500
+$Comp
+L Connector:Jack-DC J?
+U 1 1 5BD21882
+P 1650 2950
+F 0 "J?" H 1705 3275 50  0000 C CNN
+F 1 "Jack-DC" H 1705 3184 50  0000 C CNN
+F 2 "" H 1700 2910 50  0001 C CNN
+F 3 "~" H 1700 2910 50  0001 C CNN
+	1    1650 2950
 	1    0    0    -1
 $EndComp
 $Comp
-L taobao-r:R511 R?
-U 1 1 5BC25737
-P 1950 3200
-F 0 "R?" H 2050 3250 50  0000 L CNN
-F 1 "R511" H 2050 3200 50  0000 L CNN
-F 2 "" H 1950 3200 50  0001 C CNN
-F 3 "~" H 1950 3200 50  0001 C CNN
-	1    1950 3200
+L power:GND #PWR?
+U 1 1 5BD21E18
+P 2050 3150
+F 0 "#PWR?" H 2050 2900 50  0001 C CNN
+F 1 "GND" H 2055 2977 50  0000 C CNN
+F 2 "" H 2050 3150 50  0001 C CNN
+F 3 "" H 2050 3150 50  0001 C CNN
+	1    2050 3150
 	1    0    0    -1
 $EndComp
 Wire Wire Line
-	1950 2850 1950 3100
+	1950 3050 2050 3050
 Wire Wire Line
-	1950 3300 1950 3550
+	2050 3050 2050 3150
 $Comp
-L taobao-r:R102 R?
-U 1 1 5BC258E4
-P 1450 3200
-F 0 "R?" H 1550 3250 50  0000 L CNN
-F 1 "R102" H 1550 3200 50  0000 L CNN
-F 2 "" H 1450 3200 50  0001 C CNN
-F 3 "~" H 1450 3200 50  0001 C CNN
-	1    1450 3200
+L taobao-components:VIN_STM32 #PWR?
+U 1 1 5BD21FCB
+P 3300 2900
+F 0 "#PWR?" H 3300 2750 50  0001 C CNN
+F 1 "VIN_STM32" V 3305 2978 50  0000 L CNN
+F 2 "" H 3300 2900 50  0001 C CNN
+F 3 "" H 3300 2900 50  0001 C CNN
+	1    3300 2900
+	0    1    1    0
+$EndComp
+$Comp
+L taobao-components:VIN_GPS #PWR?
+U 1 1 5BD220D3
+P 3300 3300
+F 0 "#PWR?" H 3300 3150 50  0001 C CNN
+F 1 "VIN_GPS" V 3305 3378 50  0000 L CNN
+F 2 "" H 3300 3300 50  0001 C CNN
+F 3 "" H 3300 3300 50  0001 C CNN
+	1    3300 3300
+	0    1    1    0
+$EndComp
+$Comp
+L taobao-components:VIN_GSM #PWR?
+U 1 1 5BD221D8
+P 3350 3750
+F 0 "#PWR?" H 3350 3600 50  0001 C CNN
+F 1 "VIN_GSM" V 3355 3828 50  0000 L CNN
+F 2 "" H 3350 3750 50  0001 C CNN
+F 3 "" H 3350 3750 50  0001 C CNN
+	1    3350 3750
+	0    1    1    0
+$EndComp
+Wire Wire Line
+	1950 2850 2150 2850
+Wire Wire Line
+	2350 2850 2350 2900
+Connection ~ 2350 3300
+Wire Wire Line
+	2350 3300 2350 3750
+Connection ~ 2350 2900
+Wire Wire Line
+	2350 2900 2350 3300
+$Comp
+L Device:Jumper_NO_Small JP?
+U 1 1 5BD232BF
+P 2800 2900
+F 0 "JP?" H 2800 3085 50  0000 C CNN
+F 1 "Jumper_NO_Small" H 2800 2994 50  0000 C CNN
+F 2 "" H 2800 2900 50  0001 C CNN
+F 3 "~" H 2800 2900 50  0001 C CNN
+	1    2800 2900
+	1    0    0    -1
+$EndComp
+$Comp
+L Device:Jumper_NO_Small JP?
+U 1 1 5BD23305
+P 2800 3300
+F 0 "JP?" H 2800 3485 50  0000 C CNN
+F 1 "Jumper_NO_Small" H 2800 3394 50  0000 C CNN
+F 2 "" H 2800 3300 50  0001 C CNN
+F 3 "~" H 2800 3300 50  0001 C CNN
+	1    2800 3300
+	1    0    0    -1
+$EndComp
+$Comp
+L Device:Jumper_NO_Small JP?
+U 1 1 5BD2332B
+P 2800 3750
+F 0 "JP?" H 2800 3935 50  0000 C CNN
+F 1 "Jumper_NO_Small" H 2800 3844 50  0000 C CNN
+F 2 "" H 2800 3750 50  0001 C CNN
+F 3 "~" H 2800 3750 50  0001 C CNN
+	1    2800 3750
 	1    0    0    -1
 $EndComp
 Wire Wire Line
-	1450 2850 1450 3100
+	2350 3750 2700 3750
 Wire Wire Line
-	1450 3300 1450 3550
+	2900 3750 3350 3750
+Wire Wire Line
+	2350 3300 2700 3300
+Wire Wire Line
+	2900 3300 3300 3300
+Wire Wire Line
+	2350 2900 2700 2900
+Wire Wire Line
+	2900 2900 3300 2900
+$Comp
+L power:+5V #PWR?
+U 1 1 5BD24CF1
+P 2150 2750
+F 0 "#PWR?" H 2150 2600 50  0001 C CNN
+F 1 "+5V" H 2200 2950 50  0000 C CNN
+F 2 "" H 2150 2750 50  0001 C CNN
+F 3 "" H 2150 2750 50  0001 C CNN
+	1    2150 2750
+	1    0    0    -1
+$EndComp
+Wire Wire Line
+	2150 2750 2150 2850
+Connection ~ 2150 2850
+Wire Wire Line
+	2150 2850 2350 2850
 $EndSCHEMATC

Commit message: updte
Parts:
- J7: renamed from J?; footprint (none) -> footprint-lib:CUI-PJ-102A_dc-barrel-jack
- JP15, JP16, JP9: renamed from JP?; footprint (none) -> Jumper:SolderJumper-2_P1.3mm_Open_TrianglePad1.0x1.5mm
- R1: renamed from R?; footprint (none) -> Resistor_SMD:R_0805_2012Metric_Pad1.15x1.40mm_HandSolder
Changed lines of the file:
@@
 $EndComp
 $Comp
-L taobao-r:R102 R?
+L taobao-r:R102 R1
 U 1 1 5BC258E4
 P 1000 4150
-F 0 "R?" H 1100 4200 50  0000 L CNN
+F 0 "R1" H 1100 4200 50  0000 L CNN
 F 1 "R102" H 1100 4150 50  0000 L CNN
-F 2 "" H 1000 4150 50  0001 C CNN
+F 2 "Resistor_SMD:R_0805_2012Metric_Pad1.15x1.40mm_HandSolder" H 1000 4150 50  0001 C CNN
 F 3 "~" H 1000 4150 50  0001 C CNN
 	1    1000 4150
@@
 	1000 4250 1000 4500
 $Comp
-L Connector:Jack-DC J?
+L Connector:Jack-DC J7
 U 1 1 5BD21882
 P 1650 2950
-F 0 "J?" H 1705 3275 50  0000 C CNN
+F 0 "J7" H 1705 3275 50  0000 C CNN
 F 1 "Jack-DC" H 1705 3184 50  0000 C CNN
-F 2 "" H 1700 2910 50  0001 C CNN
+F 2 "footprint-lib:CUI-PJ-102A_dc-barrel-jack" H 1700 2910 50  0001 C CNN
 F 3 "~" H 1700 2910 50  0001 C CNN
 	1    1650 2950
@@
 	2350 2900 2350 3300
 $Comp
-L Device:Jumper_NO_Small JP?
+L Device:Jumper_NO_Small JP9
 U 1 1 5BD232BF
 P 2800 2900
-F 0 "JP?" H 2800 3085 50  0000 C CNN
+F 0 "JP9" H 2800 3085 50  0000 C CNN
 F 1 "Jumper_NO_Small" H 2800 2994 50  0000 C CNN
-F 2 "" H 2800 2900 50  0001 C CNN
+F 2 "Jumper:SolderJumper-2_P1.3mm_Open_TrianglePad1.0x1.5mm" H 2800 2900 50  0001 C CNN
 F 3 "~" H 2800 2900 50  0001 C CNN
 	1    2800 2900
@@
 $EndComp
 $Comp
-L Device:Jumper_NO_Small JP?
+L Device:Jumper_NO_Small JP15
 U 1 1 5BD23305
 P 2800 3300
-F 0 "JP?" H 2800 3485 50  0000 C CNN
+F 0 "JP15" H 2800 3485 50  0000 C CNN
 F 1 "Jumper_NO_Small" H 2800 3394 50  0000 C CNN
-F 2 "" H 2800 3300 50  0001 C CNN
+F 2 "Jumper:SolderJumper-2_P1.3mm_Open_TrianglePad1.0x1.5mm" H 2800 3300 50  0001 C CNN
 F 3 "~" H 2800 3300 50  0001 C CNN
 	1    2800 3300
@@
 $EndComp
 $Comp
-L Device:Jumper_NO_Small JP?
+L Device:Jumper_NO_Small JP16
 U 1 1 5BD2332B
 P 2800 3750
-F 0 "JP?" H 2800 3935 50  0000 C CNN
+F 0 "JP16" H 2800 3935 50  0000 C CNN
 F 1 "Jumper_NO_Small" H 2800 3844 50  0000 C CNN
-F 2 "" H 2800 3750 50  0001 C CNN
+F 2 "Jumper:SolderJumper-2_P1.3mm_Open_TrianglePad1.0x1.5mm" H 2800 3750 50  0001 C CNN
 F 3 "~" H 2800 3750 50  0001 C CNN
 	1    2800 3750

Commit message: updte
Parts:
- added C23: C106, Capacitor_SMD:C_0805_2012Metric_Pad1.15x1.40mm_HandSolder, symbol taobao-c:C106
- added D13: LED_ORANGE, LED_SMD:LED_0805_2012Metric_Castellated, symbol taobao-components:LED_GREEN
- added D14: 5V_STATUS, LED_SMD:LED_0805_2012Metric_Pad1.15x1.40mm_HandSolder, symbol Device:LED
- added J?: Conn_01x02, symbol Connector_Generic:Conn_01x02
- added R21, R23: R102, Resistor_SMD:R_0805_2012Metric_Pad1.15x1.40mm_HandSolder, symbol taobao-r:R102
- added R22: R222, Resistor_SMD:R_0805_2012Metric_Pad1.15x1.40mm_HandSolder, symbol taobao-r:R222
- added U14: MCP73831, Package_TO_SOT_SMD:SOT-23-5_HandSoldering, symbol taobao-components:MCP73831
Connections:
- net GND: now also C23.2, D14.1 (K), J?.2 (Pin_2), R22.2, U14.2 (VSS)
- net +5V renamed VBAT
- net VBAT: now also C23.1, J?.1 (Pin_1), U14.3 (VBAT); no longer J7.1
- new net: D13.1 (K), R21.2
- new net: R21.1, U14.1 (STAT)
- new net: R22.1, U14.5 (PROG)
- new net: D14.2 (A), R23.2
- new net VBUS: D13.2 (A), J7.1, R23.1, U14.4 (VDD)
Other:
- moved on the sheet: D12, J7, JP15, JP16, JP9, R1

Commit message: updte
Parts:
- added C24: C106, Capacitor_SMD:C_0805_2012Metric_Pad1.15x1.40mm_HandSolder, symbol taobao-c:C106
- added D15: MBR120, Diode_SMD:D_SOD-123F, symbol taobao-components:MBR120
- added U15: USB_PCB, footprint-lib:usb-PCB, symbol taobao-components:USB_PCB
- D12: value 5V_STATUS -> VBAT_STATUS
- D14: value 5V_STATUS -> VBUS_STATUS
- J12: renamed from J?; footprint (none) -> Connector_PinHeader_2.54mm:PinHeader_1x02_P2.54mm_Vertical
Connections:
- net GND: now also C24.2, U15.4 (GND)
- net VBAT: now also D15.2 (A); no longer JP15.1, JP16.1, JP9.1
- net VBUS: now also JP15.1, JP16.1, JP9.1, C24.1, D15.1 (K), U15.1 (VCC)
Other:
- moved on the sheet: C23, D13, JP15, JP16, JP9, R21, R22, U14
