File: PCB/stm32.sch (KiCad schematic (older format))
At the start: 38 parts, among them J1 Conn_01x04, J2 Conn_01x08, J3 Conn_01x08, J4 Conn_02x04_Row_Letter_First, J5 Conn_01x02, J6 Conn_01x08, J7 Conn_01x08, SW1 SW_SPST, U1 AMS1117-1.8, U2 STM32L011K4Tx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

Commit message: update
Parts:
- removed BEAD1: L1, Inductor_SMD:L_0805_2012Metric_Pad1.15x1.40mm_HandSolder, symbol Device:L
- removed C5: 100n, Capacitor_SMD:C_0603_1608Metric_Pad1.05x0.95mm_HandSolder, symbol Device:C
- removed J7: Conn_01x08, Connector_PinHeader_1.27mm:PinHeader_1x08_P1.27mm_Vertical, symbol Connector_Generic:Conn_01x08
- removed JP10, JP11, JP8, JP9: Jumper, Jumper:SolderJumper-2_P1.3mm_Bridged_Pad1.0x1.5mm, symbol Device:Jumper
- removed R4: R, Resistor_SMD:R_0805_2012Metric_Pad1.15x1.40mm_HandSolder, symbol Device:R
- removed SW1: SW_SPST, Button_Switch_THT:SW_PUSH_6mm_H4.3mm, symbol Switch:SW_SPST
- removed U2: STM32L011K4Tx, Package_QFP:LQFP-32_7x7mm_P0.8mm, symbol MCU_ST_STM32L0:STM32L011K4Tx
- added C11: 104, symbol Device:C
- added JP10, JP11, JP13, JP14: Jumper_NC_Small, symbol Device:Jumper_NC_Small
- added JP12, JP17, JP4: Jumper, symbol Device:Jumper_NC_Small
- added L2: BEAD, symbol Device:L
- added R21: 103, Resistor_SMD:R_0805_2012Metric_Pad1.15x1.40mm_HandSolder, symbol Device:R
- added SW1: SW_Push, w_switch:PCB_PUSH, symbol Switch:SW_Push
- added U2: STM32_MCU_LQFP32_QFN32, symbol taobao-components:STM32_MCU_LQFP32_QFN32
- C1: value 10u -> 56u
- C3, C4: value 4.3p -> 430
- C6, C7: value 100n -> 104
- J1: value Conn_01x04 -> PWR_CONN
- J4: value Conn_02x04_Row_Letter_First -> SWD_CONN
- J5: footprint Connector_PinHeader_2.54mm:PinHeader_1x02_P2.54mm_Vertical -> (none)
- JP1, JP2, JP3, JP5: symbol Device:Jumper -> Device:Jumper_NC_Small
- JP6: renamed from JP4; symbol Device:Jumper -> Device:Jumper_NO_Small
- JP7: renamed from JP6; symbol Device:Jumper -> Device:Jumper_NC_Small
- JP8: renamed from JP7; symbol Device:Jumper -> Device:Jumper_NO_Small
- R1, R3: value 510 -> 511
- R2: value 510 -> 102
Connections:
- net labels added: 3V3, PF0, PF1, VDD_STM32
- net labels removed: +5V
- wire segments 168 -> 166
- no-connect marks 8 -> 2
Other:
- note added: "MCO ignored"
- note removed: "MCO neglected"
- moved on the sheet: C1, C2, C3, C4, C6, C7, C8, D1, D2, D3, J1, J2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

Commit message: update
Parts:
- removed C11: 104, symbol Device:C
- removed C3, C4: 430, Capacitor_SMD:C_0603_1608Metric_Pad1.05x0.95mm_HandSolder, symbol Device:C
- removed C6, C7: 104, Capacitor_SMD:C_0603_1608Metric_Pad1.05x0.95mm_HandSolder, symbol Device:C
- removed C8: 100n, Capacitor_SMD:C_0603_1608Metric_Pad1.05x0.95mm_HandSolder, symbol Device:C
- removed D1: LED, LED_SMD:LED_0805_2012Metric_Pad1.15x1.40mm_HandSolder, symbol Device:LED
- removed D2, D3: RED, LED_SMD:LED_0805_2012Metric_Pad1.15x1.40mm_HandSolder, symbol Device:LED
- removed L2: BEAD, symbol Device:L
- removed R1, R3: 511, Resistor_SMD:R_0805_2012Metric_Pad1.15x1.40mm_HandSolder, symbol Device:R
- removed R2: 102, Resistor_SMD:R_0805_2012Metric_Pad1.15x1.40mm_HandSolder, symbol Device:R
- removed R21: 103, Resistor_SMD:R_0805_2012Metric_Pad1.15x1.40mm_HandSolder, symbol Device:R
- removed Y1: 32.768K, Crystal:Crystal_HC49-4H_Vertical, symbol Device:Crystal
- added C? (x4): C104, symbol taobao-c:C104
- added C? (x2): 430, symbol Device:C_Small
- added D? (x3): LED_Small, symbol Device:LED_Small
- added L?: BEAD, symbol Device:L_Small
- added R? (x2): R511, symbol taobao-r:R511
- added R?: R102, symbol taobao-r:R102
- added R?: R103, symbol taobao-r:R103
- added Y?: 32.768K, symbol Device:Crystal_Small
Connections:
- net labels added: +3V3
- net labels removed: 3V3

Commit message: updte
Parts:
- added D?: LED_GREEN, symbol taobao-components:LED_GREEN
- added R?: R511, symbol taobao-r:R511
- U1: value AMS1117-1.8 -> AMS1117-3.3
Connections:
- net GND: now also D?.1 (K)
- net VDD_STM32: now also R?.1
- net VIN: no longer C1.1, JP2.1, U1.3 (VI)
- new net: D?.2 (A), R?.2
- new net VIN_STM32: C1.1, JP2.1, U1.3 (VI)
Changed lines of the file:
@@
 P 2750 3700
 F 0 "U1" H 2750 3942 50  0000 C CNN
-F 1 "AMS1117-1.8" H 2750 3851 50  0000 C CNN
+F 1 "AMS1117-3.3" H 2750 3851 50  0000 C CNN
 F 2 "Package_TO_SOT_SMD:SOT-223-3_TabPin2" H 2750 3900 50  0001 C CNN
 F 3 "http://www.advanced-monolithic.com/pdf/ds1117.pdf" H 2850 3450 50  0001 C CNN
@@
 	1    0    0    -1
 $EndComp
-Text Notes 2200 3150 0    50   ~ 0
-Assuming:\n\nVIN = +5V\nVDD = +1.8V\n\n
 Wire Wire Line
 	11000 4050 11350 4050
@@
 	4950 3700 4950 3650
 $Comp
-L taobao-components:VIN #PWR0183
-U 1 1 5C0569A2
-P 1700 3650
-F 0 "#PWR0183" H 1700 3500 50  0001 C CNN
-F 1 "VIN" H 1705 3773 50  0000 C CNN
-F 2 "" H 1700 3650 50  0001 C CNN
-F 3 "" H 1700 3650 50  0001 C CNN
-	1    1700 3650
-	1    0    0    -1
-$EndComp
-$Comp
-L taobao-components:VIN #PWR0184
-U 1 1 5C056D62
-P 2150 5600
-F 0 "#PWR0184" H 2150 5450 50  0001 C CNN
-F 1 "VIN" H 2155 5723 50  0000 C CNN
-F 2 "" H 2150 5600 50  0001 C CNN
-F 3 "" H 2150 5600 50  0001 C CNN
-	1    2150 5600
-	1    0    0    -1
-$EndComp
-$Comp
 L taobao-components:VIN #PWR0186
 U 1 1 5C06D566
@@
 Wire Wire Line
 	9150 3900 9300 3900
+Text Notes 2200 3150 0    50   ~ 0
+Assuming:\n\nVIN = +5V\nVDD = +1.8V\n\n
+$Comp
+L taobao-components:VIN_STM32 #PWR?
+U 1 1 5BD1F61F
+P 2150 5600
+F 0 "#PWR?" H 2150 5450 50  0001 C CNN
+F 1 "VIN_STM32" H 2155 5723 50  0000 C CNN
+F 2 "" H 2150 5600 50  0001 C CNN
+F 3 "" H 2150 5600 50  0001 C CNN
+	1    2150 5600
+	1    0    0    -1
+$EndComp
+$Comp
+L taobao-components:VIN_STM32 #PWR?
+U 1 1 5BD1F957
+P 1700 3650
+F 0 "#PWR?" H 1700 3500 50  0001 C CNN
+F 1 "VIN_STM32" H 1705 3773 50  0000 C CNN
+F 2 "" H 1700 3650 50  0001 C CNN
+F 3 "" H 1700 3650 50  0001 C CNN
+	1    1700 3650
+	1    0    0    -1
+$EndComp
+$Comp
+L taobao-components:VDD_STM32 #PWR?
+U 1 1 5BD2515B
+P 6350 3050
+F 0 "#PWR?" H 6350 2900 50  0001 C CNN
+F 1 "VDD_STM32" H 6400 3250 50  0000 C CNN
+F 2 "" H 6350 3050 50  0001 C CNN
+F 3 "" H 6350 3050 50  0001 C CNN
+	1    6350 3050
+	1    0    0    -1
+$EndComp
+$Comp
+L taobao-r:R511 R?
+U 1 1 5BD25242
+P 6350 3300
+F 0 "R?" H 6409 3346 50  0000 L CNN
+F 1 "R511" H 6409 3255 50  0000 L CNN
+F 2 "" H 6350 3300 50  0001 C CNN
+F 3 "~" H 6350 3300 50  0001 C CNN
+	1    6350 3300
+	1    0    0    -1
+$EndComp
+$Comp
+L taobao-components:LED_GREEN D?
+U 1 1 5BD253C8
+P 6350 3650
+F 0 "D?" V 6396 3582 50  0000 R CNN
+F 1 "LED_GREEN" V 6305 3582 50  0000 R CNN
+F 2 "" V 6350 3650 50  0001 C CNN
+F 3 "~" V 6350 3650 50  0001 C CNN
+	1    6350 3650
+	0    -1   -1   0
+$EndComp
+$Comp
+L power:GND #PWR?
+U 1 1 5BD25590
+P 6350 3850
+F 0 "#PWR?" H 6350 3600 50  0001 C CNN
+F 1 "GND" H 6355 3677 50  0000 C CNN
+F 2 "" H 6350 3850 50  0001 C CNN
+F 3 "" H 6350 3850 50  0001 C CNN
+	1    6350 3850
+	1    0    0    -1
+$EndComp
+Wire Wire Line
+	6350 3750 6350 3850
+Wire Wire Line
+	6350 3400 6350 3550
+Wire Wire Line
+	6350 3050 6350 3200
 $EndSCHEMATC

Commit message: updte
Parts:
- removed C? (x2): 430, symbol Device:C_Small
- removed J4: SWD_CONN, Connector_PinHeader_2.54mm:PinHeader_2x04_P2.54mm_Vertical, symbol Connector_Generic:Conn_02x04_Row_Letter_First
- removed L?: BEAD, symbol Device:L_Small
- removed U2: STM32_MCU_LQFP32_QFN32, symbol taobao-components:STM32_MCU_LQFP32_QFN32
- removed Y?: 32.768K, symbol Device:Crystal_Small
- added C3, C4: C4.7pf, Capacitor_SMD:C_0805_2012Metric_Pad1.15x1.40mm_HandSolder, symbol taobao-c:C4.7pf
- added FB1: Ferrite_Bead_Small, w_smd_inductors:inductor_smd_0805, symbol taobao-bead:Ferrite_Bead_Small
- added J4: Conn_02x04_Odd_Even, Connector_PinHeader_2.54mm:PinHeader_2x04_P2.54mm_Vertical, symbol Connector_Generic:Conn_02x04_Odd_Even
- added U2: STM32L011K4Tx, Package_QFP:LQFP-32_7x7mm_P0.8mm, symbol taobao-components:STM32L011K4Tx
- added Y1: O32.768K, Crystal:Crystal_C38-LF_D3.0mm_L8.0mm_Vertical, symbol taobao-osc:O32.768K
- C5, C6, C7, C8: renamed from C?; footprint (none) -> Capacitor_SMD:C_0805_2012Metric_Pad1.15x1.40mm_HandSolder
- D1, D2, D3, D4: renamed from D?; footprint (none) -> LED_SMD:LED_0805_2012Metric_Castellated
- J1: footprint Connector_PinHeader_1.27mm:PinHeader_1x04_P1.27mm_Vertical -> Connector_PinHeader_2.54mm:PinHeader_1x04_P2.54mm_Vertical
- J2, J3, J6: footprint Connector_PinHeader_1.27mm:PinHeader_1x08_P1.27mm_Vertical -> Connector_PinHeader_2.54mm:PinHeader_1x08_P2.54mm_Vertical
- J5: footprint (none) -> Connector_PinHeader_2.54mm:PinHeader_1x02_P2.54mm_Vertical
- JP10, JP11, JP12, JP13, JP14, JP17, JP4: footprint (none) -> Jumper:SolderJumper-2_P1.3mm_Bridged_Pad1.0x1.5mm
- JP6, JP8: footprint Jumper:SolderJumper-2_P1.3mm_Bridged_Pad1.0x1.5mm -> Jumper:SolderJumper-2_P1.3mm_Open_TrianglePad1.0x1.5mm
- R2, R3, R4, R5, R6: renamed from R?; footprint (none) -> Resistor_SMD:R_0805_2012Metric_Pad1.15x1.40mm_HandSolder
Connections:
- net AVDD: now also FB1.2, U2.5 (VDDA/VREF+)
- net GND: now also C3.2, C4.2, J4.5 (Pin_5), J4.6 (Pin_6)
- net NRST: now also J4.8 (Pin_8), U2.4 (NRST)
- net PA0: now also U2.6 (PA0)
- net PA1: now also U2.7 (PA1)
- net PA10: now also U2.20 (PA10)
- net PA11: now also U2.21 (PA11)
- net PA12: now also U2.22 (PA12)
- net PA13: now also J4.7 (Pin_7), U2.23 (PA13)
- net PA14: now also J4.3 (Pin_3), U2.24 (PA14)
- net PA15: now also U2.25 (PA15)
- net PA2: now also U2.8 (PA2)
- net PA3: now also U2.9 (PA3)
- net PA4: now also U2.10 (PA4)
- net PA5: now also U2.11 (PA5)
- net PA6: now also U2.12 (PA6)
- net PA7: now also U2.13 (PA7)
- net PA8: now also U2.18 (PA8)
- net PA9: now also U2.19 (PA9)
- net PB0: now also U2.14 (PB0)
- net PB1: now also U2.15 (PB1/NPOR)
- net PB3: now also U2.26 (PB3)
- net PB4: now also U2.27 (PB4)
- net PB5: now also U2.28 (PB5)
- net PB6: now also U2.29 (PB6)
- net PB7: now also U2.30 (PB7)
- net VDD: now also J4.1 (Pin_1), J4.2 (Pin_2)
- net VDD_STM32: now also U2.1 (VDD3), U2.17 (VDD2/VDD_USB)
- net at JP5.1: now also C3.1, Y1.1
- net at JP4.2, JP5.2, JP6.2: now also U2.2 (PF0/PC14)
- net at JP7.1: now also C4.1, Y1.2
- net at JP7.2, JP8.2: now also U2.3 (PF1/PC15)
- net at JP11.1: now also U2.16 (PB2/VSS2)
- net at JP12.1: now also U2.31 (BOOT0/PB8/PH3)
- net at JP13.1: now also U2.32 (PB8/VSS3)
- net at JP10.1: now also FB1.1

Commit message: updte
Parts:
- D1: value LED_Small -> PB3
- D2: value LED_Small -> VIN_STATUS
- D3: value LED_Small -> VDD_STATUS
Changed lines of the file:
@@
 P 1300 7000
 F 0 "D1" V 1350 6900 50  0000 R CNN
-F 1 "LED_Small" V 1300 6900 50  0000 R CNN
+F 1 "PB3" V 1300 6900 50  0000 R CNN
 F 2 "LED_SMD:LED_0805_2012Metric_Castellated" V 1300 7000 50  0001 C CNN
 F 3 "~" V 1300 7000 50  0001 C CNN
@@
 P 2150 7000
 F 0 "D2" V 2200 6900 50  0000 R CNN
-F 1 "LED_Small" V 2150 6900 50  0000 R CNN
+F 1 "VIN_STATUS" V 2150 6900 50  0000 R CNN
 F 2 "LED_SMD:LED_0805_2012Metric_Castellated" V 2150 7000 50  0001 C CNN
 F 3 "~" V 2150 7000 50  0001 C CNN
@@
 P 3000 7000
 F 0 "D3" V 3050 6900 50  0000 R CNN
-F 1 "LED_Small" V 3000 6900 50  0000 R CNN
+F 1 "VDD_STATUS" V 3000 6900 50  0000 R CNN
 F 2 "LED_SMD:LED_0805_2012Metric_Castellated" V 3000 7000 50  0001 C CNN
 F 3 "~" V 3000 7000 50  0001 C CNN
