File: PCB/SIM800C.sch (KiCad schematic (older format))
At the start: 53 parts, among them J10 Conn_01x02, J11 USB_B_Micro, J12 TO_DTE (+3V3), J13 TO_DTE (+3V3), J14 SIM_COM_MODULE, J8 Conn_Coaxial, J9 Conn_01x02, Q1 Q_NPN_BCE, SW2 SW_SPST, U3 SIM800C, U4 MCP73831-2-OT, U5 Molex 91228 SIM card holder, U6 SMF05C

Commit message: update
Parts:
- removed C10, C13: 10u, Capacitor_SMD:C_0603_1608Metric_Pad1.05x0.95mm_HandSolder, symbol Device:C
- removed C11: 33p, Capacitor_SMD:C_0603_1608Metric_Pad1.05x0.95mm_HandSolder, symbol Device:C
- removed C12: 10p, Capacitor_SMD:C_0603_1608Metric_Pad1.05x0.95mm_HandSolder, symbol Device:C
- removed C14: 10u, Capacitor_SMD:C_0603_1608Metric_Pad1.05x0.95mm_HandSolder, symbol Device:CP
- removed C15: 1u, Capacitor_SMD:C_0603_1608Metric_Pad1.05x0.95mm_HandSolder, symbol Device:C
- removed C16: 0.1u, Capacitor_SMD:C_0603_1608Metric_Pad1.05x0.95mm_HandSolder, symbol Device:C
- removed C9: 100u, Capacitor_SMD:C_0603_1608Metric_Pad1.05x0.95mm_HandSolder, symbol Device:CP
- removed D4: MMSZ5231BT1G, Diode_SMD:D_0805_2012Metric_Pad1.15x1.40mm_HandSolder, symbol Device:D_Schottky
- removed D5, D6: D_Zener, Diode_SMD:D_0805_2012Metric_Pad1.15x1.40mm_HandSolder, symbol Device:D_Zener
- removed D7: BLUE, LED_SMD:LED_0805_2012Metric_Pad1.15x1.40mm_HandSolder, symbol Device:LED
- removed D8: GREEN, LED_SMD:LED_0805_2012Metric_Pad1.15x1.40mm_HandSolder, symbol Device:LED
- removed D_CHRG1: O, LED_SMD:LED_0805_2012Metric_Pad1.15x1.40mm_HandSolder, symbol Device:LED
- removed D_DONE1: G, LED_SMD:LED_0805_2012Metric_Pad1.15x1.40mm_HandSolder, symbol Device:LED
- removed J10, J9: Conn_01x02, Connector_PinHeader_2.54mm:PinHeader_1x02_P2.54mm_Vertical, symbol Connector_Generic:Conn_01x02
- removed J11: USB_B_Micro, Connector_USB:USB_Micro-B_Molex_47346-0001, symbol Connector:USB_B_Micro
- removed J12: TO_DTE (+3V3), Connector_PinHeader_2.54mm:PinHeader_1x05_P2.54mm_Vertical, symbol Connector_Generic:Conn_01x05
- removed J13: TO_DTE (+3V3), Connector_PinHeader_2.54mm:PinHeader_1x08_P2.54mm_Vertical, symbol Connector_Generic:Conn_01x08
- removed J14: SIM_COM_MODULE, Connector_PinHeader_2.54mm:PinHeader_1x08_P2.54mm_Vertical, symbol Connector_Generic:Conn_01x08
- removed J8: Conn_Coaxial, Connector_Coaxial:U.FL_Hirose_U.FL-R-SMT-1_Vertical, symbol Connector:Conn_Coaxial
- removed JP12: Jumper, Jumper:SolderJumper-2_P1.3mm_Bridged_Pad1.0x1.5mm, symbol Device:Jumper
- removed Q1: Q_NPN_BCE, Package_TO_SOT_SMD:SOT-23, symbol Device:Q_NPN_BCE
- removed R10, R17, R9: R, Resistor_SMD:R_0805_2012Metric_Pad1.15x1.40mm_HandSolder, symbol Device:R
- removed R11: 47k, Resistor_SMD:R_0805_2012Metric_Pad1.15x1.40mm_HandSolder, symbol Device:R
- removed R12: 10k, Resistor_SMD:R_0805_2012Metric_Pad1.15x1.40mm_HandSolder, symbol Device:R
- removed R13, R14, R15, R16, R18, R19, R23, R24, R6: 1k, Resistor_SMD:R_0805_2012Metric_Pad1.15x1.40mm_HandSolder, symbol Device:R
- removed R20, R21, R22: 5.6k, Resistor_SMD:R_0805_2012Metric_Pad1.15x1.40mm_HandSolder, symbol Device:R
- removed R25, R8: 4.7k, Resistor_SMD:R_0805_2012Metric_Pad1.15x1.40mm_HandSolder, symbol Device:R
- removed R26, R27, R28: 51, Resistor_SMD:R_0805_2012Metric_Pad1.15x1.40mm_HandSolder, symbol Device:R
- removed R5: 470, Resistor_SMD:R_0805_2012Metric_Pad1.15x1.40mm_HandSolder, symbol Device:R
- removed R7: 2k, Resistor_SMD:R_0805_2012Metric_Pad1.15x1.40mm_HandSolder, symbol Device:R
- removed SW2: SW_SPST, Button_Switch_THT:SW_PUSH_6mm_H4.3mm, symbol Switch:SW_SPST
- removed U3: SIM800C, SIMCOM_modules:SIM800C, symbol taobao-components:SIM800C
- removed U4: MCP73831-2-OT, Package_TO_SOT_SMD:SOT-23-5, symbol Battery_Management:MCP73831-2-OT
- removed U5: Molex 91228 SIM card holder, footprint-lib.pretty:sim-socket-91228-3001, symbol SIM_SLOT:SIM_CARD
- removed U6: SMF05C, w_smd_trans:sot23-6l, symbol taobao-components:SMF05C
- added C? (x2): C33pf, symbol taobao_c:C33pf
- added C?: C104, symbol taobao_c:C104
- added C?: C, symbol Device:C
- added C?: C106, symbol taobao-components:C106
- added C?: CP100u, symbol taobao-components:CP100u
- added C?: C22pf, symbol taobao_c:C22pf
- added D?: LED, symbol Device:LED
- added J? (x3): Conn_01x05, symbol Connector_Generic:Conn_01x05
- added R? (x3): R220, symbol taobao-r:R220
- added R?: R, symbol Device:R
- added R?: R102, symbol GSM-GPS-tryout-rescue:R102-taobao-components
- added U?: SMF05C, symbol taobao-components:SMF05C
- added U?: SIM_CARD, symbol SIM_SLOT:SIM_CARD
- added U?: MIC29302BU, symbol taobao-components:MIC29302BU
- added U?: SIM800C, symbol taobao-components:SIM800C
Connections:
- net labels added: ADC, BT_ANT, CTS, DCD, DN-, DP+, DTR, MICN, MICP, NET, POWER, POWERKEY, RF_SYNC, RI, RTS, RXD, RXD2, SIMVCC, SPKN, SPKP, SRXD, STA, STXD, TXD, TXD2, VDD_EXT, VDD_SIM800C, VRTC, V_MCU
- net labels removed: +1V8, +2V8, +5V, +BATT, MIC1N, MIC1P, NETLIGHT, PWRKEY, SIM800C_ADC, SIMCOM_PWRKEY, SIMDET, SPK1N, SPK1P, UART1_CTS_3V3, UART1_DCD_3V3, UART1_DTR_3V3, UART1_RI_3V3, UART1_RTS_3V3, UART1_RXD_3V3, UART1_TXD_3V3, USB_DN, USB_DP, USB_ID
- wire segments 232 -> 111
Other:
- note removed: "4.1. Power Supply"
- note removed: "COMMENTS\n\ntry to align PIN1 the GROUND\n\n4.1.1. Power Supply Pin\nThe PCB traces from the VBAT pins to the power supply must be wide enough (at least 60mil) to decrease voltage drops\nThe power IC and the bypass capacitor should be placed to the module as close as possible.\n\n4.2.1. Power on SIM800C\nCustomer can power on SIM800C by pulling down the PWRKEY pin for at least 1 second and releas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"
- note removed: "IO PORT BANK"
- note removed: "POWER SUPPLY\nAND GOUND"
- note removed: "SIM CARD HOLDER\n"
- note removed: "STATUS LED\n"
- note removed: "USB source\nand charging circuit"
- note removed: "VBAT input, a 100uF Tantalum capacitor (C A low ESR) and \na 1uF~10uF Ceramics capacitor C B are strongly recommended."
- note removed: "from SIM800C_Hardware_Design_V1.00"

Commit message: update
Parts:
- removed C? (x2): C33pf, symbol taobao_c:C33pf
- removed C?: C104, symbol taobao_c:C104
- removed C?: C106, symbol taobao-components:C106
- removed C?: CP100u, symbol taobao-components:CP100u
- removed C?: C22pf, symbol taobao_c:C22pf
- removed D?: LED, symbol Device:LED
- removed R?: R, symbol Device:R
- removed R?: R102, symbol GSM-GPS-tryout-rescue:R102-taobao-components
- added C? (x2): C33pf, symbol taobao-c:C33pf
- added C?: C22pf, symbol taobao-c:C22pf
- added C?: C104, symbol taobao-c:C104
- added C? (x2): C106, symbol taobao-c:C106
- added C?: CP_220uf, symbol taobao-cp:CP_220uf
- added C?: CP_100uf, symbol taobao-cp:CP_100uf
- added D?: D_Zener_Small, symbol Device:D_Zener_Small
- added D?: LED_Small, symbol Device:LED_Small
- added R? (x2): R102, symbol taobao-r:R102
- added R?: R433, symbol taobao-r:R433
- added R?: R104, symbol taobao-r:R104
- added R?: R471, symbol taobao-r:R471
- added R?: R_Small, symbol Device:R_Small
Connections:
- wire segments 111 -> 146

Commit message: updte
Parts:
- removed C?: C, symbol Device:C
- removed C?: CP_220uf, symbol taobao-cp:CP_220uf
- removed C?: CP_100uf, symbol taobao-cp:CP_100uf
- removed D?: LED_Small, symbol Device:LED_Small
- added C?: TC107,6V, symbol taobao-tc:TC107,6V
- added C?: C106, symbol taobao-c:C106
- added C?: CP220uf,16V, symbol taobao-cp:CP220uf,16V
- added C?: C104, symbol taobao-c:C104
- added D?: LED_GREEN, symbol taobao-components:LED_GREEN
- added D?: LED_RED, symbol taobao-components:LED_RED
- added J?: Conn_01x02, symbol Connector_Generic:Conn_01x02
- added U?: GSM_SMA, w_conn_rf:sma_straight_32k101-400l5, symbol taobao-components:SMA
- added U?: BT_SMA, w_conn_rf:sma_straight_32k101-400l5, symbol taobao-components:SMA
- added U?: USB_PCB, symbol taobao-components:USB_PCB
Connections:
- net labels added: BT_ANT_GND, DP-, GSM_ANT_GND
- wire segments 146 -> 173
Other:
- moved on the sheet: C?, D?, R?

Commit message: updte
Connections:
- net VDD_SIM800C: now also C?.1, C?.1, D?.1 (K), R?.1, R?.1, R?.2, U?.4 (OUT)
- net POWER renamed VIN_GSM
Changed lines of the file:
@@
 Wire Wire Line
 	2950 7150 2950 7200
-Text Label 2800 7050 2    50   ~ 0
-POWER
 Wire Wire Line
 	2800 7050 2250 7050
@@
 	1    0    0    -1
 $EndComp
-Text Label 11350 7600 0    50   ~ 0
-POWER
 Wire Wire Line
 	11350 7600 11850 7600
@@
 	13900 7950 13900 8250
 Wire Wire Line
-	14250 7600 14550 7600
+	14250 7600 14450 7600
 $Comp
 L taobao-c:C106 C?
@@
 	13900 4800 14400 4800
 Connection ~ 14400 4800
+$Comp
+L taobao-components:VIN_GSM #PWR?
+U 1 1 5BD0E615
+P 2800 7000
+F 0 "#PWR?" H 2800 6850 50  0001 C CNN
+F 1 "VIN_GSM" H 2805 7123 50  0000 C CNN
+F 2 "" H 2800 7000 50  0001 C CNN
+F 3 "" H 2800 7000 50  0001 C CNN
+	1    2800 7000
+	1    0    0    -1
+$EndComp
+$Comp
+L taobao-components:VIN_GSM #PWR?
+U 1 1 5BD0E9B6
+P 11350 7550
+F 0 "#PWR?" H 11350 7400 50  0001 C CNN
+F 1 "VIN_GSM" H 11355 7673 50  0000 C CNN
+F 2 "" H 11350 7550 50  0001 C CNN
+F 3 "" H 11350 7550 50  0001 C CNN
+	1    11350 7550
+	1    0    0    -1
+$EndComp
+Wire Wire Line
+	11350 7550 11350 7600
+Wire Wire Line
+	2800 7000 2800 7050
+$Comp
+L taobao-components:VDD_SIM800C #PWR?
+U 1 1 5BD4537B
+P 14450 7500
+F 0 "#PWR?" H 14450 7350 50  0001 C CNN
+F 1 "VDD_SIM800C" H 14467 7673 50  0000 C CNN
+F 2 "" H 14450 7500 50  0001 C CNN
+F 3 "" H 14450 7500 50  0001 C CNN
+	1    14450 7500
+	1    0    0    -1
+$EndComp
+Wire Wire Line
+	14450 7500 14450 7600
+Connection ~ 14450 7600
+Wire Wire Line
+	14450 7600 14550 7600
 $EndSCHEMATC

Commit message: updte
Parts:
- added D?: LED_GREEN, symbol taobao-components:LED_GREEN
- added R?: R102, symbol taobao-r:R102
Connections:
- net GND: now also D?.1 (K)
- net VDD_SIM800C: now also R?.1
- new net: D?.2 (A), R?.2
Changed lines of the file:
@@
 	8650 3850 9800 3850
 $Comp
-L power:GND #PWR?
+L power:GND #PWR0130
 U 1 1 5C1742BF
 P 8950 4350
-F 0 "#PWR?" H 8950 4100 50  0001 C CNN
+F 0 "#PWR0130" H 8950 4100 50  0001 C CNN
 F 1 "GND" V 8955 4222 50  0000 R CNN
 F 2 "" H 8950 4350 50  0001 C CNN
@@
 	9150 4750 9800 4750
 $Comp
-L power:GND #PWR?
+L power:GND #PWR0131
 U 1 1 5C1745F0
 P 8700 4950
-F 0 "#PWR?" H 8700 4700 50  0001 C CNN
+F 0 "#PWR0131" H 8700 4700 50  0001 C CNN
 F 1 "GND" H 8705 4777 50  0000 C CNN
 F 2 "" H 8700 4950 50  0001 C CNN
@@
 	10700 5250 10700 5800
 $Comp
-L power:GND #PWR?
+L power:GND #PWR0132
 U 1 1 5BC1D87E
 P 10450 5500
-F 0 "#PWR?" H 10450 5250 50  0001 C CNN
+F 0 "#PWR0132" H 10450 5250 50  0001 C CNN
 F 1 "GND" V 10455 5372 50  0000 R CNN
 F 2 "" H 10450 5500 50  0001 C CNN
@@
 	11000 5250 11000 5800
 $Comp
-L power:GND #PWR?
+L power:GND #PWR0133
 U 1 1 5BC1E1CB
 P 11400 5600
-F 0 "#PWR?" H 11400 5350 50  0001 C CNN
+F 0 "#PWR0133" H 11400 5350 50  0001 C CNN
 F 1 "GND" H 11405 5427 50  0000 C CNN
 F 2 "" H 11400 5600 50  0001 C CNN
@@
 	12500 4100 11800 4100
 $Comp
-L power:GND #PWR?
+L power:GND #PWR0134
 U 1 1 5BC23495
 P 12400 3550
-F 0 "#PWR?" H 12400 3300 50  0001 C CNN
+F 0 "#PWR0134" H 12400 3300 50  0001 C CNN
 F 1 "GND" H 12405 3377 50  0000 C CNN
 F 2 "" H 12400 3550 50  0001 C CNN
@@
 	12500 3800 11800 3800
 $Comp
-L power:GND #PWR?
+L power:GND #PWR0135
 U 1 1 5BC24F8A
 P 12100 4000
-F 0 "#PWR?" H 12100 3750 50  0001 C CNN
+F 0 "#PWR0135" H 12100 3750 50  0001 C CNN
 F 1 "GND" V 12105 3872 50  0000 R CNN
 F 2 "" H 12100 4000 50  0001 C CNN
@@
 	11300 2950 11400 2950
 $Comp
-L power:GND #PWR?
+L power:GND #PWR0136
 U 1 1 5BC3A8D2
 P 11850 2750
-F 0 "#PWR?" H 11850 2500 50  0001 C CNN
+F 0 "#PWR0136" H 11850 2500 50  0001 C CNN
 F 1 "GND" V 11855 2622 50  0000 R CNN
 F 2 "" H 11850 2750 50  0001 C CNN
@@
 $EndComp
 $Comp
-L taobao-components:VDD_SIM800C #PWR?
+L taobao-components:VDD_SIM800C #PWR0137
 U 1 1 5BC3AA63
 P 11300 2350
-F 0 "#PWR?" H 11300 2200 50  0001 C CNN
+F 0 "#PWR0137" H 11300 2200 50  0001 C CNN
 F 1 "VDD_SIM800C" H 11317 2523 50  0000 C CNN
 F 2 "" H 11300 2350 50  0001 C CNN
@@
 Connection ~ 11750 2750
 $Comp
-L power:GND #PWR?
+L power:GND #PWR0138
 U 1 1 5BC4009B
 P 11050 2850
-F 0 "#PWR?" H 11050 2600 50  0001 C CNN
+F 0 "#PWR0138" H 11050 2600 50  0001 C CNN
 F 1 "GND" H 11055 2677 50  0000 C CNN
 F 2 "" H 11050 2850 50  0001 C CNN
@@
 	10800 2600 10800 3250
 $Comp
-L power:GND #PWR?
+L power:GND #PWR0139
 U 1 1 5BC43B8A
 P 10800 2250
-F 0 "#PWR?" H 10800 2000 50  0001 C CNN
+F 0 "#PWR0139" H 10800 2000 50  0001 C CNN
 F 1 "GND" H 10805 2077 50  0000 C CNN
 F 2 "" H 10800 2250 50  0001 C CNN
@@
 	10700 2700 10700 3250
 $Comp
-L power:GND #PWR?
+L power:GND #PWR0140
 U 1 1 5BC49A6A
 P 9700 2600
-F 0 "#PWR?" H 9700 2350 50  0001 C CNN
+F 0 "#PWR0140" H 9700 2350 50  0001 C CNN
 F 1 "GND" H 9705 2427 50  0000 C CNN
 F 2 "" H 9700 2600 50  0001 C CNN
@@
 	14650 1000 14900 1000
 $Comp
-L power:GND #PWR?
+L power:GND #PWR0141
 U 1 1 5BC5647D
 P 15350 1100
-F 0 "#PWR?" H 15350 850 50  0001 C CNN
+F 0 "#PWR0141" H 15350 850 50  0001 C CNN
 F 1 "GND" H 15355 927 50  0000 C CNN
 F 2 "" H 15350 1100 50  0001 C CNN
@@
 $EndComp
 $Comp
-L power:GND #PWR?
+L power:GND #PWR0142
 U 1 1 5BC63449
 P 8150 8250
-F 0 "#PWR?" H 8150 8000 50  0001 C CNN
+F 0 "#PWR0142" H 8150 8000 50  0001 C CNN
 F 1 "GND" H 8155 8077 50  0000 C CNN
 F 2 "" H 8150 8250 50  0001 C CNN
@@
 $EndComp
 $Comp
-L power:GND #PWR?
+L power:GND #PWR0143
 U 1 1 5BC30AC7
 P 5400 7450
-F 0 "#PWR?" H 5400 7200 50  0001 C CNN
+F 0 "#PWR0143" H 5400 7200 50  0001 C CNN
 F 1 "GND" H 5405 7277 50  0000 C CNN
 F 2 "" H 5400 7450 50  0001 C CNN
@@
 Connection ~ 5400 7350
 $Comp
-L power:GND #PWR?
+L power:GND #PWR0144
 U 1 1 5BC3625C
 P 6500 6050
-F 0 "#PWR?" H 6500 5800 50  0001 C CNN
+F 0 "#PWR0144" H 6500 5800 50  0001 C CNN
 F 1 "GND" V 6505 5922 50  0000 R CNN
 F 2 "" H 6500 6050 50  0001 C CNN
@@
 Connection ~ 6100 7550
 $Comp
-L power:GND #PWR?
+L power:GND #PWR0145
 U 1 1 5BC54C0A
 P 6100 7900
-F 0 "#PWR?" H 6100 7650 50  0001 C CNN
+F 0 "#PWR0145" H 6100 7650 50  0001 C CNN
 F 1 "GND" H 6105 7727 50  0000 C CNN
 F 2 "" H 6100 7900 50  0001 C CNN
@@
 $EndComp
 $Comp
-L power:GND #PWR?
+L power:GND #PWR0146
 U 1 1 5BC581D3
 P 8500 6700
-F 0 "#PWR?" H 8500 6450 50  0001 C CNN
+F 0 "#PWR0146" H 8500 6450 50  0001 C CNN
 F 1 "GND" H 8505 6527 50  0000 C CNN
 F 2 "" H 8500 6700 50  0001 C CNN
@@
 	2800 7250 2250 7250
 $Comp
-L power:GND #PWR?
+L power:GND #PWR0147
 U 1 1 5BC6A221
 P 2950 7200
-F 0 "#PWR?" H 2950 6950 50  0001 C CNN
+F 0 "#PWR0147" H 2950 6950 50  0001 C CNN
 F 1 "GND" H 2955 7027 50  0000 C CNN
 F 2 "" H 2950 7200 50  0001 C CNN
@@
 Connection ~ 12450 8500
 $Comp
-L power:GND #PWR?
+L power:GND #PWR0148
 U 1 1 5BC6A9E0
 P 12550 8650
-F 0 "#PWR?" H 12550 8400 50  0001 C CNN
+F 0 "#PWR0148" H 12550 8400 50  0001 C CNN
 F 1 "GND" H 12600 8450 50  0000 C CNN
 F 2 "" H 12550 8650 50  0001 C CNN
@@
 $EndComp
 $Comp
-L power:GND #PWR?
+L power:GND #PWR0149
 U 1 1 5BC76624
 P 14300 5400
-F 0 "#PWR?" H 14300 5150 50  0001 C CNN
+F 0 "#PWR0149" H 14300 5150 50  0001 C CNN
 F 1 "GND" V 14305 5272 50  0000 R CNN
 F 2 "" H 14300 5400 50  0001 C CNN
@@
 $EndComp
 $Comp
-L taobao-components:VDD_SIM800C #PWR?
+L taobao-components:VDD_SIM800C #PWR0150
 U 1 1 5BC7DEDF
 P 14300 5500
-F 0 "#PWR?" H 14300 5350 50  0001 C CNN
+F 0 "#PWR0150" H 14300 5350 50  0001 C CNN
 F 1 "VDD_SIM800C" V 14318 5628 50  0000 L CNN
 F 2 "" H 14300 5500 50  0001 C CNN
@@
 	13900 4050 14450 4050
 $Comp
-L power:GND #PWR?
+L power:GND #PWR0151
 U 1 1 5BCD9549
 P 14400 4300
-F 0 "#PWR?" H 14400 4050 50  0001 C CNN
+F 0 "#PWR0151" H 14400 4050 50  0001 C CNN
 F 1 "GND" H 14405 4127 50  0000 C CNN
 F 2 "" H 14400 4300 50  0001 C CNN
@@
 	13900 4650 14450 4650
 $Comp
-L power:GND #PWR?
+L power:GND #PWR0152
 U 1 1 5BCE8D0E
 P 14400 4900
-F 0 "#PWR?" H 14400 4650 50  0001 C CNN
+F 0 "#PWR0152" H 14400 4650 50  0001 C CNN
 F 1 "GND" H 14405 4727 50  0000 C CNN
 F 2 "" H 14400 4900 50  0001 C CNN
@@
 Connection ~ 14400 4800
 $Comp
-L taobao-components:VIN_GSM #PWR?
+L taobao-components:VIN_GSM #PWR0153
 U 1 1 5BD0E615
 P 2800 7000
-F 0 "#PWR?" H 2800 6850 50  0001 C CNN
+F 0 "#PWR0153" H 2800 6850 50  0001 C CNN
 F 1 "VIN_GSM" H 2805 7123 50  0000 C CNN
 F 2 "" H 2800 7000 50  0001 C CNN
@@
 $EndComp
 $Comp
-L taobao-components:VIN_GSM #PWR?
+L taobao-components:VIN_GSM #PWR0154
 U 1 1 5BD0E9B6
 P 11350 7550
-F 0 "#PWR?" H 11350 7400 50  0001 C CNN
+F 0 "#PWR0154" H 11350 7400 50  0001 C CNN
 F 1 "VIN_GSM" H 11355 7673 50  0000 C CNN
 F 2 "" H 11350 7550 50  0001 C CNN
@@
 	2800 7000 2800 7050
 $Comp
-L taobao-components:VDD_SIM800C #PWR?
+L taobao-components:VDD_SIM800C #PWR0155
 U 1 1 5BD4537B
 P 14450 7500
-F 0 "#PWR?" H 14450 7350 50  0001 C CNN
+F 0 "#PWR0155" H 14450 7350 50  0001 C CNN
 F 1 "VDD_SIM800C" H 14467 7673 50  0000 C CNN
 F 2 "" H 14450 7500 50  0001 C CNN
@@
 Wire Wire Line
 	14450 7600 14550 7600
+$Comp
+L taobao-components:VDD_SIM800C #PWR0156
+U 1 1 5BD4DFE2
+P 2650 2300
+F 0 "#PWR0156" H 2650 2150 50  0001 C CNN
+F 1 "VDD_SIM800C" H 2667 2473 50  0000 C CNN
+F 2 "" H 2650 2300 50  0001 C CNN
+F 3 "" H 2650 2300 50  0001 C CNN
+	1    2650 2300
+	1    0    0    -1
+$EndComp
+$Comp
+L taobao-r:R102 R?
+U 1 1 5BD4E13F
+P 2650 2550
+F 0 "R?" H 2709 2596 50  0000 L CNN
+F 1 "R102" H 2709 2505 50  0000 L CNN
+F 2 "" H 2650 2550 50  0001 C CNN
+F 3 "~" H 2650 2550 50  0001 C CNN
+	1    2650 2550
+	1    0    0    -1
+$EndComp
+$Comp
+L taobao-components:LED_GREEN D?
+U 1 1 5BD4E2FC
+P 2650 2900
+F 0 "D?" V 2696 2832 50  0000 R CNN
+F 1 "LED_GREEN" V 2605 2832 50  0000 R CNN
+F 2 "" V 2650 2900 50  0001 C CNN
+F 3 "~" V 2650 2900 50  0001 C CNN
+	1    2650 2900
+	0    -1   -1   0
+$EndComp
+$Comp
+L power:GND #PWR0157
+U 1 1 5BD4E448
+P 2650 3150
+F 0 "#PWR0157" H 2650 2900 50  0001 C CNN
+F 1 "GND" H 2655 2977 50  0000 C CNN
+F 2 "" H 2650 3150 50  0001 C CNN
+F 3 "" H 2650 3150 50  0001 C CNN
+	1    2650 3150
+	1    0    0    -1
+$EndComp
+Wire Wire Line
+	2650 2300 2650 2450
+Wire Wire Line
+	2650 2650 2650 2800
+Wire Wire Line
+	2650 3000 2650 3150
 $EndSCHEMATC

Commit message: updte
Parts:
- removed D?: D_Zener_Small, symbol Device:D_Zener_Small
- removed U?: SIM_CARD, symbol SIM_SLOT:SIM_CARD
- added D7: ZD_4V7, Diode_SMD:D_1206_3216Metric_Pad1.42x1.75mm_HandSolder, symbol taobao-zd:ZD_4V7
- added U3: footprint-lib_nano-sim-card-holder, footprint-lib:nano-sim-card-holder, symbol taobao-components:footprint-lib_nano-sim-card-holder
- C10, C11, C12, C14, C15, C9: renamed from C?; footprint (none) -> Capacitor_SMD:C_0805_2012Metric_Pad1.15x1.40mm_HandSolder
- C13: renamed from C?; footprint (none) -> Capacitor_Tantalum_SMD:CP_EIA-3216-12_Kemet-S_Pad1.58x1.35mm_HandSolder
- C16: renamed from C?; footprint (none) -> Capacitor_SMD:CP_Elec_6.3x7.7
- C17, C18: renamed from C?; footprint (none) -> Capacitor_SMD:C_0603_1608Metric_Pad1.05x0.95mm_HandSolder
- D5, D6, D8: renamed from D?; footprint (none) -> LED_SMD:LED_0805_2012Metric_Castellated
- J10, J8, J9: renamed from J?; footprint (none) -> Connector_PinHeader_2.54mm:PinHeader_1x05_P2.54mm_Vertical
- J11: renamed from J?; footprint (none) -> Connector_PinHeader_2.54mm:PinHeader_1x02_P2.54mm_Vertical
- R10, R11, R12, R13, R14, R15, R16, R7, R8, R9: renamed from R?; footprint (none) -> Resistor_SMD:R_0805_2012Metric_Pad1.15x1.40mm_HandSolder
- U12: renamed from U?; footprint (none) -> footprint-lib:usb-PCB
- U4: renamed from U?; footprint (none) -> Package_TO_SOT_SMD:SOT-363_SC-70-6_Handsoldering
- U5: renamed from U?; footprint (none) -> footprint-lib:LCC110P1570X1760X250-42N
- U6: renamed from U?; footprint (none) -> Package_TO_SOT_SMD:TO-263-5_TabPin3
- gave numbers to parts that had none: 2
Connections:
- net GND: now also U3.2 (GND1)
- net SIMVCC: now also U3.1 (VCC)
- net VDD_SIM800C: now also D7.1 (K)
- net at R8.1, U4.4: now also U3.3 (RST)
- net at R9.1, U4.3: now also U3.5 (CLK)
- net at R10.1, U4.6: now also U3.6 (I/O)
- net at C16.2, C17.2, D8.1 (K)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: now also D7.2 (A)

Commit message: updte
Parts:
- removed U12: USB_PCB, footprint-lib:usb-PCB, symbol taobao-components:USB_PCB
- added J13: SIM800_DEBUG, w_conn_pc:conn_usb_B_micro_smd, symbol Connector:USB_B_Micro
Connections:
- net DP+: now also J13.3 (D+)
- net DP-: now also J13.2 (D-)
- net GND: now also J13.5 (GND), J13.6 (Shield)
- net USB_VBUS: now also J13.1 (VBUS)
Changed lines of the file:
@@
 	15000 8250 15000 8000
 Connection ~ 14550 8250
-$Comp
-L taobao-components:USB_PCB U12
-U 1 1 5BD538D1
-P 14850 6050
-F 0 "U12" H 15177 6121 50  0000 L CNN
-F 1 "USB_PCB" H 15177 6030 50  0000 L CNN
-F 2 "footprint-lib:usb-PCB" H 14850 6100 50  0001 C CNN
-F 3 "" H 14850 6100 50  0001 C CNN
-	1    14850 6050
-	1    0    0    -1
-$EndComp
-Text Label 13900 5900 0    50   ~ 0
+Text Label 14050 5900 0    50   ~ 0
 USB_VBUS
 Wire Wire Line
-	13900 5900 14500 5900
-Text Label 13900 6100 0    50   ~ 0
+	14050 5900 14650 5900
+Text Label 14050 6100 0    50   ~ 0
 DP+
 Wire Wire Line
-	13900 6100 14500 6100
-Text Label 13900 6000 0    50   ~ 0
+	14050 6100 14650 6100
+Text Label 14050 6200 0    50   ~ 0
 DP-
 Wire Wire Line
-	13900 6000 14500 6000
-Text Label 13900 6200 0    50   ~ 0
+	14050 6200 14650 6200
+Text Label 14200 6550 0    50   ~ 0
 GND
-Wire Wire Line
-	13900 6200 14500 6200
 $Comp
 L taobao-tc:TC107,6V C13
@@
 	0    1    1    0
 $EndComp
+$Comp
+L Connector:USB_B_Micro J13
+U 1 1 5BC7E777
+P 14950 6100
+F 0 "J13" H 14720 6091 50  0000 R CNN
+F 1 "SIM800_DEBUG" H 14720 6000 50  0000 R CNN
+F 2 "w_conn_pc:conn_usb_B_micro_smd" H 15100 6050 50  0001 C CNN
+F 3 "~" H 15100 6050 50  0001 C CNN
+	1    14950 6100
+	-1   0    0    -1
+$EndComp
+Wire Wire Line
+	14950 6550 14950 6500
+Wire Wire Line
+	14200 6550 14950 6550
+Wire Wire Line
+	14950 6550 15050 6550
+Wire Wire Line
+	15050 6550 15050 6500
+Connection ~ 14950 6550
 $EndSCHEMATC
