File: PCB/SIM800C.sch (KiCad schematic (older format))
At the start: 27 parts

Commit message: update,
Parts:
- C?: symbol taobao-cp:CP_220uf -> GSM-GPS-tryout-rescue:CP_220uf-taobao-cp
- C?: symbol taobao-cp:CP_100uf -> GSM-GPS-tryout-rescue:CP_100uf-taobao-cp
Changed lines of the file:
@@
 Connection ~ 13700 7600
 $Comp
-L taobao-cp:CP_220uf C?
+L GSM-GPS-tryout-rescue:CP_220uf-taobao-cp C?
 U 1 1 5BC8FB97
 P 14700 7850
@@
 	13400 4200 13650 4200
 $Comp
-L taobao-cp:CP_100uf C?
+L GSM-GPS-tryout-rescue:CP_100uf-taobao-cp C?
 U 1 1 5BD52440
 P 11500 2950
